File: PCB/mengpaneel.sch (KiCad schematic (older format))
At the start: 339 parts, among them IC1 MAX7219CNG+, IC2 MAX7219CNG+, IC3 MTCH6301-I_ML, J1 AudioJack3_Ground, J2 Screw_Terminal_01x02, J3 Screw_Terminal_01x09, SW1 SW_Push, SW2 SW_DPDT_x2, SW3 SW_DPST_x2, SW4 SW_DPST_x2, U1 OPAMP, U10 OPAMP, U11 AD5290, U12 OPAMP, U13 AD5290, U14 AD5290, U15 AD5290, U16 AD5290, U17 AD5290, U18 AD5290, U19 AD5290, U2 AD5290, U20 AD5290, U21 AD5290, U22 AD5290, U23 AD5290, U24 OPAMP, U25 OPAMP, U26 OPAMP, U27 AD5290, U28 AD5290, U29 AD5290, U3 AD5290, U31 LM3480-3.3, U32 STM32F413RGTx, U4 AD5290, U5 OPAMP, U6 AD5290, U7 OPAMP, U8 AD5290, U9 OPAMP, Y1 8MHz

Commit message: update 23/03/2021 alle libraries aangepast naar definitieve componenten
Parts:
- removed C48, C49, C51, C52, C53, C54, C55, C56, C57, C58, C61, C62, C65, C66, C67, C68, C69, C70: 20p, symbol Device:C
- removed Input1, Input2, J1, Microfoon1: AudioJack3_Ground, symbol Connector:AudioJack3_Ground
- removed R57: 100K, symbol Device:R
- removed R61, R64, R65, R66, R67, R71, R72, R73, R74, R75, R76, R78, R79, R80, R81, R82, R83, R84: 2.2k, symbol Device:R
- removed R62, R63: 4K7, symbol Device:R
- removed U11, U13, U14, U15, U16, U17, U18, U19, U2, U20, U21, U22, U23, U27, U28, U29, U3, U4, U6, U8: AD5290, Package_SO:MSOP-10_3x3mm_P0.5mm, symbol Potentiometer_Digital:AD5290
- removed U31: LM3480-3.3, Package_TO_SOT_SMD:SOT-23, symbol Regulator_Linear:LM3480-3.3
- removed U32: STM32F413RGTx, Package_QFP:LQFP-64_10x10mm_P0.5mm, symbol MCU_ST_STM32F4:STM32F413RGTx
- added C? (x2): 0.1µF, symbol Device:C
- added IC10: STM32F411CEU7, STM32F411CEU7:QFN50P700X700X65-49N-D, symbol STM32F411CEU7:STM32F411CEU7
- added IC11, IC5, IC6, IC8, IC9: AD5204BRUZ10-REEL7, SOP65P640X120-24N, symbol AD5204BRUZ10-REEL7:AD5204BRUZ10-REEL7
- added IC12: LTC3631EMS8E#TRPBF, SOP65P490X110-9N, symbol LTC3631EMS8E#TRPBF:LTC3631EMS8E#TRPBF
- added IC4: LTC3121EDE#PBF, LTC3121EDE#PBF:SON50P300X400X80-13N-D, symbol LTC3121EDE#PBF:LTC3121EDE#PBF
- added IC7: LM3480IM3-3.3_NOPB, LM3480IM3-3.3_NOPB:SOT95P237X112-3N, symbol LM3480IM3-3.3_NOPB:LM3480IM3-3.3_NOPB
- added J1: UJ2-MIBH-G-SMT-TR, UJ2-MIBH-G-SMT-TR:UJ2MIBHGSMTTR, symbol UJ2-MIBH-G-SMT-TR:UJ2-MIBH-G-SMT-TR
- added J4, J5, J6, J7: SJ-63053A, SJ-63053A:SJ63053A, symbol SJ-63053A:SJ-63053A
- added L2: 100µ, symbol Device:L
- added U30: touchpad_lib_Touchpad_mp, symbol schema_tp-cache:touchpad_lib_Touchpad_mp
- C45: value 20p -> 1µ
- C46: value 20p -> 10µ
- IC1, IC2: symbol MAX7219CNG+:MAX7219CNG+ -> mengpaneel-rescue:MAX7219CNG+-MAX7219CNG+
- IC3: symbol MTCH6301-I_ML:MTCH6301-I_ML -> mengpaneel-rescue:MTCH6301-I_ML-MTCH6301-I_ML
- R59: value 2.2k -> 1M
- R60: value 2.2k -> 71,5k
- U1: value OPAMP -> LMV321AUIDBVR
- U10, U12, U24, U25, U26, U5, U7, U9: value OPAMP -> LM324N
Connections:
- net labels added: NRST, POT10_A, POT10_B, POT10_W, POT11_A, POT11_B, POT11_W, POT12_A, POT12_B, POT12_W, POT13_A, POT13_B, POT13_W, POT14_A, POT14_B, POT14_W, POT15_A, POT15_B, POT15_W, POT16_A, POT16_B, POT16_W, POT17_A, POT17_B, POT17_W, POT18_A, POT18_W, POT19_A, POT19_B, POT1_A, POT1_W, POT20_A, POT20_W, POT2_A, POT2_W, POT3_A, POT3_W, POT4_A, POT4_W, POT5_A, POT5_W, POT6_A, POT6_B, POT6_W, POT7_A, POT7_B, POT7_W, POT8_A, POT8_B, POT8_W, POT9_A, POT9_B, POT9_W, PReset_POT, SD_POT, SD_Step-Up
- net labels removed: L1.10, L1.11, L1.12, L1.13, L1.14, L1.15, L1.16, L1.17, L1.18, L1.19, L1.20, L1.6, L1.7, L1.8, L1.9
- wire segments 1314 -> 1205
Other:
- note removed: "DIT IS DE LTC3121EDE#PBF"
- note removed: "Nog wachten op mail!"
- note removed: "dit mag weg"
- moved on the sheet: C36, C37, C38, C40, C41, C42, C43, C44, C47, C64, C71, C72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

Commit message: associatie footprint associatie footprint
Parts:
- removed U30: touchpad_lib_Touchpad_mp, symbol schema_tp-cache:touchpad_lib_Touchpad_mp
- added U11, U14, U15, U16, U17, U2, U3, U4, U6: Touchpad_mp, symbol touchpad_mengpaneel_library:Touchpad_mp
- added U13: Touchpad_mp_LR, schema_tp:touchpad_footprint_LR, symbol touchpad_mengpaneel_library:Touchpad_mp_LR
- added U8: Touchpad_mp, schema_tp:touchpad_footprint_normaal, symbol touchpad_mengpaneel_library:Touchpad_mp
- IC10: symbol STM32F411CEU7:STM32F411CEU7 -> mengpaneel-rescue:STM32F411CEU7-STM32F411CEU7
- IC11, IC5, IC6, IC8, IC9: symbol AD5204BRUZ10-REEL7:AD5204BRUZ10-REEL7 -> mengpaneel-rescue:AD5204BRUZ10-REEL7-AD5204BRUZ10-REEL7
- IC12: footprint SOP65P490X110-9N -> LTC3631EMS8E#TRPBF:SOP65P490X110-9N; symbol LTC3631EMS8E#TRPBF:LTC3631EMS8E#TRPBF -> mengpaneel-rescue:LTC3631EMS8E#TRPBF-LTC3631EMS8E#TRPBF
- IC4: symbol LTC3121EDE#PBF:LTC3121EDE#PBF -> mengpaneel-rescue:LTC3121EDE#PBF-LTC3121EDE#PBF
- IC7: symbol LM3480IM3-3.3_NOPB:LM3480IM3-3.3_NOPB -> mengpaneel-rescue:LM3480IM3-3.3_NOPB-LM3480IM3-3.3_NOPB
- J1: symbol UJ2-MIBH-G-SMT-TR:UJ2-MIBH-G-SMT-TR -> mengpaneel-rescue:UJ2-MIBH-G-SMT-TR-UJ2-MIBH-G-SMT-TR
- J4, J5, J6, J7: symbol SJ-63053A:SJ-63053A -> mengpaneel-rescue:SJ-63053A-SJ-63053A
- gave numbers to parts that had none: 2
Connections:
- net labels removed: Slider_1x, Slider_2x, Slider_3x
- wire segments 1205 -> 1160

Commit message: 23/03/2021 verdere aanpassing
Parts:
- removed J2: Screw_Terminal_01x02, symbol Connector:Screw_Terminal_01x02
- removed J3: Screw_Terminal_01x09, symbol Connector:Screw_Terminal_01x09
- added J2: Screw_Terminal_01x03, symbol Connector:Screw_Terminal_01x03
- added J3: Screw_Terminal_01x14, symbol Connector:Screw_Terminal_01x14
Connections:
- net labels added: CS_POT1, CS_POT2, CS_POT3, CS_POT4, CS_POT5, I2C_SCL, I2C_SDA, SPI1_MOSI, SPI1_SCK, SPI2_MOSI, SPI2_SCK, UART_CLK, laag1_1, laag1_10, laag1_11, laag1_12, laag1_2, laag1_3, laag1_4, laag1_5, laag1_6, laag1_7, laag1_8, laag1_9, laag2_1, laag2_10, laag2_11, laag2_12, laag2_2, laag2_3, laag2_4, laag2_5, laag2_6, laag2_7, laag2_8, laag2_9, laag3_1, laag3_10, laag3_11, laag3_12, laag3_2, laag3_3, laag3_4, laag3_5, laag3_6, laag3_7, laag3_8, laag3_9, laag4_1, laag4_10, laag4_11, laag4_12, laag4_2, laag4_3, laag4_4, laag4_5, laag4_6, laag4_7, laag4_8, laag4_9
- net labels removed: CS_POT, CS_POT_mic, Din1_POT, Din_Leds, L1.1, L1.2, L1.3, L1.4, L1.5, Slider_10.1, Slider_10.10, Slider_10.11, Slider_10.12, Slider_10.2, Slider_10.3, Slider_10.4, Slider_10.5, Slider_10.6, Slider_10.7, Slider_10.8, Slider_10.9, Slider_10x, Slider_11.1, Slider_11.10, Slider_11.11, Slider_11.12, Slider_11.2, Slider_11.3, Slider_11.4, Slider_11.5, Slider_11.6, Slider_11.7, Slider_11.8, Slider_11.9, Slider_11x, Slider_4.1, Slider_4.10, Slider_4.11, Slider_4.12, Slider_4.2, Slider_4.3, Slider_4.4, Slider_4.5, Slider_4.6, Slider_4.7, Slider_4.8, Slider_4.9, Slider_4x, Slider_5.1, Slider_5.10, Slider_5.11, Slider_5.12, Slider_5.2, Slider_5.3, Slider_5.4, Slider_5.5, Slider_5.6, Slider_5.7, Slider_5.8, Slider_5.9, Slider_5x, Slider_6.1, Slider_6.10, Slider_6.11, Slider_6.12, Slider_6.2, Slider_6.3, Slider_6.4, Slider_6.5, Slider_6.6, Slider_6.7, Slider_6.8, Slider_6.9, Slider_6x, Slider_7.1, Slider_7.10, Slider_7.11, Slider_7.12, Slider_7.2, Slider_7.3, Slider_7.4, Slider_7.5, Slider_7.6, Slider_7.7, Slider_7.8, Slider_7.9, Slider_7x, Slider_8.1, Slider_8.10, Slider_8.11, Slider_8.12, Slider_8.2, Slider_8.3, Slider_8.4, Slider_8.5, Slider_8.6, Slider_8.7, Slider_8.8, Slider_8.9, Slider_8x, Slider_9.1, Slider_9.10, Slider_9.11, Slider_9.12, Slider_9.2, Slider_9.3, Slider_9.4, Slider_9.5, Slider_9.6, Slider_9.7, Slider_9.8, Slider_9.9, Slider_9x
- wire segments 1160 -> 1100
- no-connect marks 58 -> 72
Other:
- note added: "L-R"
- note removed: "L-R Line 1"
- moved on the sheet: SW2A, SW3A, SW3B, SW4A, U11, U13, U14, U15, U16, U17, U2, U3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

Commit message: tussentijdse vernieuwing 27/03/2021
Parts:
- removed U1: LMV321AUIDBVR, symbol pspice:OPAMP
- removed U10, U12, U24, U25, U26, U5, U7, U9: LM324N, symbol pspice:OPAMP
- added C51: C1206C100K5RACTU, C1206C100K5RACTU:CAPC3216X88N, symbol C1206C100K5RACTU:C1206C100K5RACTU
- added IC13: LMV321AUIDBVR, SOT95P280X145-5N, symbol LMV321AUIDBVR:LMV321AUIDBVR
- added U5, U7: LM324N, LM324N:DIP794W56P254L1905H533Q14N, symbol Amplifier_Operational:LM324
- C1, C11, C12, C15, C19, C39, C6: footprint (none) -> MAL219299601E3:CAPAE1050X1050N
- C10, C21, C22, C23, C24, C25, C26, C9: footprint (none) -> EMF212B7225KGHT:CAPC2012X135N
- C13, C28, C29, C32: footprint (none) -> C0805F682K1RACAUTO:CAPC2012X100N
- C14, C27, C30, C31: footprint (none) -> C0402C152J3GACAUTO:CAPC1005X55N
- C16, C18, C20, C8: footprint (none) -> EEE-FK1K4R7V:CAPAE660X610N
- C17, C2, C3, C33, C34, C35, C4, C45, C5, C7: footprint (none) -> C0805X105K8RAC7210:CAPC2012X100N
- C36, C37, C48, C49: value 0.1µF -> 0.1µ; footprint (none) -> 06031C104K4Z2A:CAPC1608X90N
- C38, C40: footprint (none) -> JMK212B7475KGHT:CAPC2114X145N
- C41: value 150p -> 390p; footprint (none) -> C0603C391J1HACTU:CAPC1608X87N
- C42: value 100nF -> 100n
- C44: footprint (none) -> C1206C100K5RACTU:CAPC3216X88N
- C46, C50: footprint (none) -> TMK212BC6106KG-T:CAPC2114X145N
- C47, C64: footprint (none) -> C0402C180F5GACTU:CAPC1005X55N
- C59, C60, C63, C72, C73: footprint (none) -> 06031C104K4Z2A:CAPC1608X90N
- C71: footprint (none) -> C0805C226K7PACTU:CAPC2012X140N
- D1, D100, D109, D110, D111, D112, D121, D122, D123, D124, D13, D14, D15, D16, D2, D25, D26, D27, D28, D3, D37, D38, D39, D4, D40, D49, D50, D51, D52, D61, D62, D63, D64, D73, D74, D75, D76, D85, D86, D87, D88, D97, D98, D99: footprint (none) -> 598-8C10-107F:LEDM2214X135N
- D10, D105, D106, D107, D108, D11, D117, D118, D119, D12, D120, D129, D130, D131, D132, D21, D22, D23, D24, D33, D34, D35, D36, D45, D46, D47, D48, D57, D58, D59, D60, D69, D70, D71, D72, D81, D82, D83, D84, D9, D93, D94, D95, D96: footprint (none) -> 598-8C80-107F:LEDM2214X135N
- D101, D102, D103, D104, D113, D114, D115, D116, D125, D126, D127, D128, D17, D18, D19, D20, D29, D30, D31, D32, D41, D42, D43, D44, D5, D53, D54, D55, D56, D6, D65, D66, D67, D68, D7, D77, D78, D79, D8, D80, D89, D90, D91, D92: footprint (none) -> 598-8C30-107F:LEDM2214X135N
- IC1, IC2: footprint (none) -> MAX7219CNG+:DIP794W56P254L3054H457Q24N
- IC3: footprint (none) -> MTCH6301-I_ML:QFN65P800X800X100-45N-D
- L1: value 6.8µH -> 6.8µ; footprint (none) -> SRP0512-6R8K:SRP05126R8K
- R1, R68, R69, R70: footprint (none) -> ERA-2VEB1001X:RESC1005X40N
- R10, R13, R15, R18, R21, R23, R24, R25, R30, R32, R33, R35, R36, R38, R39, R41, R42, R44, R45, R47: footprint (none) -> CMP2010-FX-1002ELF:RESC5025X70N
- R11, R2, R26, R28, R29, R3, R4, R5, R58, R6, R8, R9: footprint (none) -> ERJ-UP3D1003V:RESC1608X55N
- R12, R14, R16, R17, R22, R27, R31, R34, R37, R40, R43, R46, R48, R49, R50, R7: footprint (none) -> RCS120622K0JNEA:RESC3216X65N
- R19, R20: footprint (none) -> CR0805-FX-9531ELF:RESC2012X60N
- R51, R52, R53, R54: footprint (none) -> CMP2010AFX-2000ELF:RESC5025X70N
- R55, R56: footprint (none) -> CMP2010AFX-1000ELF:RESC5025X70N
- R85: footprint (none) -> CR0603-FX-5762ELF:RESC1608X55N
- R86: footprint (none) -> RQ73C2A210KBTDF:RESC2012X65N
- R87: footprint (none) -> CRCW06031M02FKEA:RESC1608X50N
- R88: footprint (none) -> CR0805-FX-1133ELF:RESC2012X60N
- U11, U14, U15, U16, U17, U2, U3, U4, U6: footprint (none) -> schema_tp:touchpad_footprint_normaal
- Y1: footprint (none) -> ECS-80-18-4X-CKM:ECS80184XCKM
Connections:
- net +12V: now also IC13.3 (+IN), U5.4 (V+), U7.4 (V+)
- net -12V: now also IC13.4 (-IN), U5.11 (V-), U7.11 (V-)
- net GND: now also IC13.5 (V+), U5.10 (+), U5.12 (+), U7.10 (+), U7.12 (+)
- net POT1_A: now also IC13.1 (OUT)
- net UART_CLK: now also J2.3 (Pin_3)
- net at R1.2, R2.1: now also IC13.2 (V-)
- net at C13.2, C14.2, R27.2: now also U5.9 (-)
- net at C17.1, R21.2, R22.2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: now also U5.8
- net at C1.2, J6.3: no longer J6.2
- net at R11.2, R13.1, R14.1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: now also U5.1
- net at R10.2, R11.1: now also U5.2 (-)
- net at C6.1: now also U5.3 (+)
- net at C31.2, C32.2, R50.2: now also U7.13 (-)
- net at C35.1, R45.2, R46.2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: now also U7.14
- net at R25.2, R29.1: now also U7.6 (-)
- net at C15.1: now also U7.5 (+)
- net at R29.2, R36.1, R37.1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: now also U7.7
- net at C29.2, C30.2, R49.2: now also U7.9 (-)
- net at C34.1, R42.2, R43.2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: now also U7.8
- net at R24.2, R28.1: now also U7.2 (-)
- net at C12.1: now also U7.3 (+)
- net at R28.2, R33.1, R34.1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: now also U7.1
- net at C27.2, C28.2, R48.2: now also U5.13 (-)
- net at C33.1, R39.2, R40.2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: now also U5.14
- net at R26.2, R30.1, R31.1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: now also U5.7
- net at R18.2, R26.1: now also U5.6 (-)
- net at C11.1: now also U5.5 (+)
- no-connect marks 72 -> 73
Other:
- note added: "groen"
- note added: "oranje"
- note added: "rood\n"

Commit message: PCB bijna af
Parts:
- removed C51: C1206C100K5RACTU, C1206C100K5RACTU:CAPC3216X88N, symbol C1206C100K5RACTU:C1206C100K5RACTU
- C42, C43: footprint (none) -> C1206C100K5RACTU:CAPC3216X88N
- D123, D124: footprint 598-8C10-107F:LEDM2214X135N -> 598-8C30-107F:LEDM2214X135N
- D125, D126, D127, D128: footprint 598-8C30-107F:LEDM2214X135N -> 598-8C80-107F:LEDM2214X135N
- D129, D130: footprint 598-8C80-107F:LEDM2214X135N -> 598-8C30-107F:LEDM2214X135N
- D131, D132: footprint 598-8C80-107F:LEDM2214X135N -> 598-8C10-107F:LEDM2214X135N
- IC11, IC5, IC6, IC8, IC9: footprint SOP65P640X120-24N -> AD5204BRUZ10-REEL7:SOP65P640X120-24N
- IC13: footprint SOT95P280X145-5N -> LMV321AUIDBVR:SOT95P280X145-5N
- J2: footprint (none) -> Connector_PinHeader_1.00mm:PinHeader_1x03_P1.00mm_Vertical
- J3: footprint (none) -> Connector_PinHeader_1.00mm:PinHeader_1x14_P1.00mm_Vertical
- L2: footprint (none) -> LQM21DN101M70L:VARC2012X145N
- R59: footprint (none) -> ERJ-UP3D1004V:RESC1608X55N
- R60: footprint (none) -> ERJ-UP3F7152V:RESC1608X55N
- R77: footprint (none) -> RCC04022K20FKED:RESC1005X40N
- SW1: footprint (none) -> PTS526_SK15_SMTR2_LFS:PTS526SK15SMTR2LFS
- SW2: footprint (none) -> Connector_PinHeader_1.00mm:PinHeader_1x06_P1.00mm_Vertical
- SW3, SW4: footprint (none) -> Connector_PinHeader_1.00mm:PinHeader_1x04_P1.00mm_Vertical
Connections:
- net POT18_W is gone; now on net GND: IC9.20 (W2)
- net POT19_B is gone; now on net GND: IC9.13 (B3)
- net SCL is gone; now on net I2C_SCL: IC3.44 (SCL), R68.2
- net SDA is gone; now on net I2C_SDA: IC3.1 (SDA), R69.2
- net GND: no longer IC9.14 (W3), IC9.21 (B2)
- net POT17_A: no longer R51.1, R52.2, R55.1, R55.2, R56.2
- net POT17_B: no longer R53.1, R54.2, R56.1
- net POT17_W: no longer C19.1, C39.1
- net POT18_A: now also R51.1, R52.2, R55.2
- net POT19_A: now also R55.1
- net POT20_A: now also R56.2
- net POT20_W: now also C39.1
- new net POT18_B: IC9.21 (B2), R53.1, R54.2, R56.1
- new net POT19_W: C19.1, IC9.14 (W3)

Commit message: PCB af alleen nog wachten op touchsliders
Parts:
- C72, C73: footprint 06031C104K4Z2A:CAPC1608X90N -> 0603YC104J4T4A:CAPC1608X90N
Connections:
- net LEDlaag_11: now also D14.2 (A), D2.2 (A), D26.2 (A), D38.2 (A)
- net laag_1: now also U13.14 (Y_00)
- net laag_10: now also U13.23 (Y_09)
- net laag_11: now also U13.24 (Y_010)
- net laag_12: now also U13.25 (Y_011)
- net laag_2: now also U13.15 (Y_01)
- net laag_3: now also U13.16 (Y_02)
- net laag_4: now also U13.17 (Y_03)
- net laag_5: now also U13.18 (Y_04)
- net laag_6: now also U13.19 (Y_05)
- net laag_7: now also U13.20 (Y_06)
- net laag_8: now also U13.21 (Y_07)
- net laag_9: now also U13.22 (Y_08)
- net laag4_1: no longer names the net of U13.2 (Y_0)
- net laag4_1: no longer U15.14 (Y_00)
- net laag4_10: no longer names the net of U13.11 (Y_9)
- net laag4_10: no longer U15.23 (Y_09)
- net laag4_11: no longer names the net of U13.12 (Y_10)
- net laag4_11: no longer U15.24 (Y_010)
- net laag4_12: no longer names the net of U13.13 (Y_11)
- net laag4_12: no longer U15.25 (Y_011)
- net laag4_2: no longer names the net of U13.3 (Y_1)
- net laag4_2: no longer U15.15 (Y_01)
- net laag4_3: no longer names the net of U13.4 (Y_2)
- net laag4_3: no longer U15.16 (Y_02)
- net laag4_4: no longer names the net of U13.5 (Y_3)
- net laag4_4: no longer U15.17 (Y_03)
- net laag4_5: no longer names the net of U13.6 (Y_4)
- net laag4_5: no longer U15.18 (Y_04)
- net laag4_6: no longer names the net of U13.7 (Y_5)
- net laag4_6: no longer U15.19 (Y_05)
- net laag4_7: no longer names the net of U13.8 (Y_6)
- net laag4_7: no longer U15.20 (Y_06)
- net laag4_8: no longer names the net of U13.9 (Y_7)
- net laag4_8: no longer U15.21 (Y_07)
- net laag4_9: no longer names the net of U13.10 (Y_8)
- net laag4_9: no longer U15.22 (Y_08)
- no-connect marks 73 -> 85
Changed lines of the file:
@@
 F 0 "C72" H 17535 15216 50  0000 L CNN
 F 1 "0,1µ" H 17535 15125 50  0000 L CNN
-F 2 "06031C104K4Z2A:CAPC1608X90N" H 17458 15020 50  0001 C CNN
+F 2 "0603YC104J4T4A:CAPC1608X90N" H 17458 15020 50  0001 C CNN
 F 3 "~" H 17420 15170 50  0001 C CNN
 	1    17420 15170
@@
 F 0 "C73" H 17535 15676 50  0000 L CNN
 F 1 "0.1µ" H 17535 15585 50  0000 L CNN
-F 2 "06031C104K4Z2A:CAPC1608X90N" H 17458 15480 50  0001 C CNN
+F 2 "0603YC104J4T4A:CAPC1608X90N" H 17458 15480 50  0001 C CNN
 F 3 "~" H 17420 15630 50  0001 C CNN
 	1    17420 15630
@@
 NoConn ~ 14880 9580
 NoConn ~ 14880 9380
-$Comp
-L touchpad_mengpaneel_library:Touchpad_mp_LR U13
-U 1 1 609ED08E
-P 6680 10900
-F 0 "U13" H 6755 11265 50  0000 C CNN
-F 1 "Touchpad_mp_LR" H 6755 11174 50  0000 C CNN
-F 2 "schema_tp:touchpad_footprint_LR" H 6680 11400 50  0001 C CNN
-F 3 "" H 6680 11400 50  0001 C CNN
-	1    6680 10900
-	1    0    0    -1
-$EndComp
 $Comp
 L touchpad_mengpaneel_library:Touchpad_mp U8
@@
 Text GLabel 4440 9180 0    50   Input ~ 0
 laag3_12
-Text GLabel 8650 10280 2    50   Input ~ 0
-laag4_1
-Text GLabel 8650 10180 2    50   Input ~ 0
-laag4_2
-Text GLabel 8650 10080 2    50   Input ~ 0
-laag4_3
-Text GLabel 8650 9980 2    50   Input ~ 0
-laag4_4
-Text GLabel 8650 9880 2    50   Input ~ 0
-laag4_5
-Text GLabel 8650 9780 2    50   Input ~ 0
-laag4_6
-Text GLabel 8650 9680 2    50   Input ~ 0
-laag4_7
-Text GLabel 8650 9580 2    50   Input ~ 0
-laag4_8
-Text GLabel 8650 9480 2    50   Input ~ 0
-laag4_9
-Text GLabel 8650 9380 2    50   Input ~ 0
-laag4_10
-Text GLabel 8650 9280 2    50   Input ~ 0
-laag4_11
-Text GLabel 8650 9180 2    50   Input ~ 0
-laag4_12
-Text GLabel 6380 11900 0    50   Input ~ 0
-laag4_1
-Text GLabel 6380 11800 0    50   Input ~ 0
-laag4_2
-Text GLabel 6380 11700 0    50   Input ~ 0
-laag4_3
-Text GLabel 6380 11600 0    50   Input ~ 0
-laag4_4
-Text GLabel 6380 11500 0    50   Input ~ 0
-laag4_5
-Text GLabel 6380 11400 0    50   Input ~ 0
-laag4_6
-Text GLabel 6380 11300 0    50   Input ~ 0
-laag4_7
-Text GLabel 6380 11200 0    50   Input ~ 0
-laag4_8
-Text GLabel 6380 11100 0    50   Input ~ 0
-laag4_9
-Text GLabel 6380 11000 0    50   Input ~ 0
-laag4_10
-Text GLabel 6380 10900 0    50   Input ~ 0
-laag4_11
-Text GLabel 6380 10800 0    50   Input ~ 0
-laag4_12
-NoConn ~ 7130 10800
-NoConn ~ 7130 10900
-NoConn ~ 7130 11000
-NoConn ~ 7130 11100
-NoConn ~ 7130 11200
-NoConn ~ 7130 11300
-NoConn ~ 7130 11400
-NoConn ~ 7130 11500
-NoConn ~ 7130 11600
-NoConn ~ 7130 11700
-NoConn ~ 7130 11800
-NoConn ~ 7130 11900
 $Comp
 L Connector:Screw_Terminal_01x03 J2
@@
 Text GLabel 23850 18970 3    35   Input ~ 0
 POT17_A
+Wire Wire Line
+	4470 13280 5060 13280
+Connection ~ 4470 13280
+Connection ~ 5060 13280
+$Comp
+L touchpad_mengpaneel_library:Touchpad_mp_LR U13
+U 1 1 609ED08E
+P 6680 10900
+F 0 "U13" H 6755 11265 50  0000 C CNN
+F 1 "Touchpad_mp_LR" H 6755 11174 50  0000 C CNN
+F 2 "schema_tp:touchpad_footprint_LR" H 6680 11400 50  0001 C CNN
+F 3 "" H 6680 11400 50  0001 C CNN
+	1    6680 10900
+	1    0    0    -1
+$EndComp
+Text GLabel 7130 11900 2    50   Input ~ 0
+laag_1
+Text GLabel 7130 11800 2    50   Input ~ 0
+laag_2
+Text GLabel 7130 11700 2    50   Input ~ 0
+laag_3
+Text GLabel 7130 11600 2    50   Input ~ 0
+laag_4
+Text GLabel 7130 11500 2    50   Input ~ 0
+laag_5
+Text GLabel 7130 11400 2    50   Input ~ 0
+laag_6
+Text GLabel 7130 11300 2    50   Input ~ 0
+laag_7
+Text GLabel 7130 11200 2    50   Input ~ 0
+laag_8
+Text GLabel 7130 11100 2    50   Input ~ 0
+laag_9
+Text GLabel 7130 11000 2    50   Input ~ 0
+laag_10
+Text GLabel 7130 10900 2    50   Input ~ 0
+laag_11
+Text GLabel 7130 10800 2    50   Input ~ 0
+laag_12
+NoConn ~ 8650 9180
+NoConn ~ 8650 9280
+NoConn ~ 8650 9380
+NoConn ~ 8650 9480
+NoConn ~ 8650 9580
+NoConn ~ 8650 9680
+NoConn ~ 8650 9780
+NoConn ~ 8650 9880
+NoConn ~ 8650 9980
+NoConn ~ 8650 10080
+NoConn ~ 8650 10180
+NoConn ~ 8650 10280
+NoConn ~ 6380 10800
+NoConn ~ 6380 10900
+NoConn ~ 6380 11000
+NoConn ~ 6380 11100
+NoConn ~ 6380 11200
+NoConn ~ 6380 11300
+NoConn ~ 6380 11400
+NoConn ~ 6380 11500
+NoConn ~ 6380 11900
+NoConn ~ 6380 11800
+NoConn ~ 6380 11700
+NoConn ~ 6380 11600
 $EndSCHEMATC
