File: PCB/mengpaneel.sch (KiCad schematic (older format))
At the start: 296 parts, among them IC1 MAX7219CNG+, IC10 STM32F411CEU7, IC11 AD5204BRUZ10-REEL7, IC12 LTC3631EMS8E#TRPBF, IC13 LMV321AUIDBVR, IC2 MAX7219CNG+, IC3 MTCH6301-I_ML, IC4 LTC3121EDE#PBF, IC5 AD5204BRUZ10-REEL7, IC6 AD5204BRUZ10-REEL7, IC8 AD5204BRUZ10-REEL7, IC9 AD5204BRUZ10-REEL7, J1 UJ2-MIBH-G-SMT-TR, J2 Screw_Terminal_01x03, J3 Screw_Terminal_01x14, J4 SJ-63053A, J5 SJ-63053A, J6 SJ-63053A, J7 SJ-63053A, SW1 SW_Push, SW2 SW_DPDT_x2, SW3 SW_DPST_x2, SW4 SW_DPST_x2, U11 Touchpad_mp, U13 Touchpad_mp_LR, U14 Touchpad_mp, U15 Touchpad_mp, U16 Touchpad_mp, U17 Touchpad_mp, U2 Touchpad_mp, U3 Touchpad_mp, U4 Touchpad_mp, U5 LM324N, U6 Touchpad_mp, U7 LM324N, U8 Touchpad_mp, Y1 8MHz

Commit message: Document beginnen invullen
Other:
- note added: "BASS LIN1"
- note added: "BASS LIN2"
- note added: "LIN1 IN"
- note added: "MASTER OUT"
- note added: "MEDIUM LIN1"
- note added: "MEDIUM LIN2"
- note added: "MICROFOON VOLUME"
- note added: "TREBLE LIN1"
- note added: "TREBLE LIN2"
- note added: "Verhoog de stroom er van.\n"
- note removed: "BASS"
- note removed: "Line 1 IN"
- note removed: "MEDIUM"
- note removed: "MICROFOON"
- note removed: "OUT"
- note removed: "TREBLE"
Changed lines of the file:
@@
 Text GLabel 9140 12780 2    50   Input ~ 0
 LEDlaag_12
-Text Notes 3670 6250 0    50   ~ 0
-BASS
-Text Notes 9210 6280 0    50   ~ 0
-BASS
-Text Notes 9240 7950 0    50   ~ 0
-MEDIUM
-Text Notes 9240 9600 0    50   ~ 0
-TREBLE
-Text Notes 3500 7960 0    50   ~ 0
-MEDIUM
-Text Notes 3450 9620 0    50   ~ 0
-TREBLE
-Text Notes 4640 3840 0    50   ~ 0
-Line 1 IN
-Text Notes 8050 3800 0    50   ~ 0
+Text Notes 3170 3820 0    50   ~ 0
+BASS LIN1
+Text Notes 9240 6280 0    50   ~ 0
+BASS LIN2
+Text Notes 3210 8140 0    50   ~ 0
+MEDIUM LIN2
+Text Notes 9200 8110 0    50   ~ 0
+TREBLE LIN2
+Text Notes 4540 3820 0    50   ~ 0
+MEDIUM LIN1
+Text Notes 7980 3800 0    50   ~ 0
+TREBLE LIN1
+Text Notes 9500 3810 0    50   ~ 0
+LIN1 IN
+Text Notes 3390 6400 0    50   ~ 0
 Line 2 IN
-Text Notes 9610 3810 0    50   ~ 0
-OUT
+Text Notes 9170 9740 0    50   ~ 0
+MASTER OUT
 Text GLabel 2990 5250 0    50   Input ~ 0
 laag_1
@@
 Text GLabel 3340 5400 2    50   Input ~ 0
 slider_1
-Text Notes 3160 3820 0    50   ~ 0
-MICROFOON
+Text Notes 2980 9770 0    50   ~ 0
+MICROFOON VOLUME
 Wire Wire Line
 	3740 4150 4420 4150
@@
 Wire Wire Line
 	16840 17420 16840 17840
+Wire Notes Line
+	14570 14260 14570 13230
+Wire Notes Line
+	14670 14260 14670 14180
+Wire Notes Line
+	14670 14180 14780 14180
+Wire Notes Line
+	14780 14180 14780 14120
+Wire Notes Line
+	14890 14120 14890 14050
+Wire Notes Line
+	14570 14260 14670 14260
+Wire Notes Line
+	14780 14120 14890 14120
+Wire Notes Line
+	14890 14050 14940 14050
+Wire Notes Line
+	14560 14260 14490 14260
+Wire Notes Line
+	14490 14260 14490 14180
+Wire Notes Line
+	14490 14180 14400 14180
+Wire Notes Line
+	14400 14180 14400 14080
+Wire Notes Line
+	14400 14080 14310 14080
+Wire Notes Line
+	14310 14080 14310 13990
+Wire Notes Line
+	14310 13990 14210 13990
+Text Notes 14190 13100 0    50   ~ 0
+Verhoog de stroom er van.\n
 $EndSCHEMATC

Commit message: PCB doet aan alle normen van de docent
Parts:
- removed C41: 390p, C0603C391J1HACTU:CAPC1608X87N, symbol Device:C
- removed C44: 10p, C1206C100K5RACTU:CAPC3216X88N, symbol Device:C
- removed C71: 22µ, C0805C226K7PACTU:CAPC2012X140N, symbol Device:C
- removed J2: Screw_Terminal_01x03, Connector_PinHeader_1.00mm:PinHeader_1x03_P1.00mm_Vertical, symbol Connector:Screw_Terminal_01x03
- removed L1: 6.8µ, SRP0512-6R8K:SRP05126R8K, symbol Device:L
- removed R86: 210k, RQ73C2A210KBTDF:RESC2012X65N, symbol Device:R
- removed R87: 1.02M, CRCW06031M02FKEA:RESC1608X50N, symbol Device:R
- removed R88: 113k, CR0805-FX-1133ELF:RESC2012X60N, symbol Device:R
- removed SW2: SW_DPDT_x2, Connector_PinHeader_1.00mm:PinHeader_1x06_P1.00mm_Vertical, symbol Switch:SW_DPDT_x2
- added C51: 4.7µ, JMK212B7475KGHT:CAPC2114X145N, symbol Device:C
- added C52: 1n, C0402C102J4GACAUTO:CAPC1005X55N, symbol Device:C
- added C53: 68p, 06035C680KAT2A:CAPC1608X90N, symbol Device:C
- added C54: 47µ, C5750X7R1C476M230KB:CAPC5750X250N, symbol Device:C
- added J10, J11, J12, J13, J14, J15, J16, J17, J2, J8, J9: Screw_Terminal_01x01, Connector_PinHeader_1.00mm:PinHeader_1x01_P1.00mm_Vertical, symbol Connector:Screw_Terminal_01x01
- added J18: Screw_Terminal_01x12, Connector_PinHeader_1.00mm:PinHeader_1x12_P1.00mm_Vertical, symbol Connector:Screw_Terminal_01x12
- added L3: 3.3µ, SPM6530T-3R3M:INDPM7165X315N, symbol Device:L
- added R57: 43.2k, CR0805-FX-4322ELF:RESC2012X60N, symbol Device:R
- added R61: 383k, CR1206-FX-3833ELF:RESC3216X75N, symbol Device:R
- added R62: 121k, CR0805-FX-1213ELF:RESC2012X60N, symbol Device:R
- added SW2: SW_DPST_x2, Connector_PinHeader_1.00mm:PinHeader_1x04_P1.00mm_Vertical, symbol Switch:SW_DPST_x2
- C72: value 0,1µ -> 0.1µ
Connections:
- net labels added: Data+, Data-, ID
- net labels removed: RX_UART, TX_UART, UART_CLK
- wire segments 1120 -> 1125
- no-connect marks 82 -> 80
Other:
- note removed: "Verhoog de stroom er van.\n"
- moved on the sheet: C40, J3, R85

Commit message: word in git steken.
Parts:
- added J?: Screw_Terminal_01x05, symbol Connector:Screw_Terminal_01x05
Connections:
- net +12V: now also C45.1, IC12.2 (VIN), IC12.5 (RUN)
- net 3.3V: now also J?.1 (Pin_1)
- net 5V: no longer C45.1, IC12.2 (VIN), IC12.5 (RUN)
- net CS_POT5: now also IC10.33 (PA12); no longer IC10.37 (PA14)
- net GND: now also J?.5 (Pin_5)
- net NRST: now also J?.4 (Pin_4)
- net SWDIO: now reaches IC10.34 (PA13)
- net SWDIO: now also J?.2 (Pin_2)
- net Data+: no longer names the net of J1.3
- net Data+: no longer IC10.33 (PA12)
- net Data-: no longer names the net of J1.2
- net Data-: no longer IC10.32 (PA11)
- net ID: no longer names the net of J1.4
- net ID: no longer IC10.31 (PA10)
- new net SWCLK: IC10.37 (PA14), J?.3 (Pin_3)
- no-connect marks 80 -> 81
Changed lines of the file:
@@
 	19270 13930 19270 13990
 Text GLabel 17960 13030 0    50   Input ~ 0
-5V
++12V
 Wire Wire Line
 	18570 13030 18450 13030
@@
 Text GLabel 16280 8580 1    50   Input ~ 0
 CS_POT4
-Text GLabel 16380 8580 1    50   Input ~ 0
+Text GLabel 16680 9580 2    50   Input ~ 0
 CS_POT5
 Text GLabel 17970 20540 0    50   Input ~ 0
@@
 NoConn ~ 7130 10900
 NoConn ~ 7130 11000
-Text Notes 17820 17240 0    50   ~ 0
+Text Notes 17880 16710 0    50   ~ 0
 Component alleen nog bestellen
 $Comp
@@
 	1    0    0    -1
 $EndComp
-Text GLabel 16680 9680 2    50   Input ~ 0
-Data-
-Text GLabel 16680 9580 2    50   Input ~ 0
-Data+
-Text GLabel 12280 13380 2    50   Input ~ 0
-Data-
-Text GLabel 12280 13080 2    50   Input ~ 0
-Data+
+Text GLabel 19650 9370 0    50   Input ~ 0
+SWCLK
+Text GLabel 19650 9170 0    50   Input ~ 0
+3.3V
 $Comp
 L Switch:SW_DPST_x2 SW2
@@
 	-1   0    0    -1
 $EndComp
-Text GLabel 16680 9780 2    50   Input ~ 0
-ID
-Text GLabel 12280 13180 2    50   Input ~ 0
-ID
-NoConn ~ 16680 9480
+Text GLabel 19650 9270 0    50   Input ~ 0
+SWDIO
 $Comp
 L Device:C C51
@@
 Wire Wire Line
 	15590 16090 15960 16090
+Text GLabel 19650 9470 0    50   Input ~ 0
+NRST
+$Comp
+L Connector:Screw_Terminal_01x05 J?
+U 1 1 614D0ABC
+P 19850 9370
+F 0 "J?" H 19930 9412 50  0000 L CNN
+F 1 "Screw_Terminal_01x05" H 19930 9321 50  0000 L CNN
+F 2 "" H 19850 9370 50  0001 C CNN
+F 3 "~" H 19850 9370 50  0001 C CNN
+	1    19850 9370
+	1    0    0    -1
+$EndComp
+Text GLabel 19650 9570 0    50   Input ~ 0
+GND
+Text GLabel 16380 8580 1    50   Input ~ 0
+SWCLK
+Text GLabel 16680 9480 2    50   Input ~ 0
+SWDIO
+NoConn ~ 16680 9680
+NoConn ~ 16680 9780
 $EndSCHEMATC

Commit message: pcb oke
Parts:
- removed C38, C40, C51: 4.7µ, JMK212B7475KGHT:CAPC2114X145N, symbol Device:C
- removed C43: 100n, C1206C100K5RACTU:CAPC3216X88N, symbol Device:C
- removed C45: 1µ, C0805X105K8RAC7210:CAPC2012X100N, symbol Device:C
- removed C46: 10µ, TMK212BC6106KG-T:CAPC2114X145N, symbol Device:C
- removed C52: 1n, C0402C102J4GACAUTO:CAPC1005X55N, symbol Device:C
- removed C53: 68p, 06035C680KAT2A:CAPC1608X90N, symbol Device:C
- removed C54: 47µ, C5750X7R1C476M230KB:CAPC5750X250N, symbol Device:C
- removed C72, C73: 0.1µ, 0603YC104J4T4A:CAPC1608X90N, symbol Device:C
- removed IC12: LTC3631EMS8E#TRPBF, LTC3631EMS8E#TRPBF:SOP65P490X110-9N, symbol mengpaneel-rescue:LTC3631EMS8E#TRPBF-LTC3631EMS8E#TRPBF
- removed IC4: LTC3121EDE#PBF, LTC3121EDE#PBF:SON50P300X400X80-13N-D, symbol mengpaneel-rescue:LTC3121EDE#PBF-LTC3121EDE#PBF
- removed L2: 100µ, LQM21DN101M70L:VARC2012X145N, symbol Device:L
- removed L3: 3.3µ, SPM6530T-3R3M:INDPM7165X315N, symbol Device:L
- removed R57: 43.2k, CR0805-FX-4322ELF:RESC2012X60N, symbol Device:R
- removed R59: 1M, ERJ-UP3D1004V:RESC1608X55N, symbol Device:R
- removed R60: 71,5k, ERJ-UP3F7152V:RESC1608X55N, symbol Device:R
- removed R61: 383k, CR1206-FX-3833ELF:RESC3216X75N, symbol Device:R
- removed R62: 121k, CR0805-FX-1213ELF:RESC2012X60N, symbol Device:R
- removed R85: 57.6k, CR0603-FX-5762ELF:RESC1608X55N, symbol Device:R
- added C41: 0.1µ, 06031C104K4Z2A:CAPC1608X90N, symbol Device:C
- added C44, C55, C56, C57, C58: 1µ, C0805X105K8RAC7210:CAPC2012X100N, symbol Device:C
- added R63, R64: 1k, ERA-2VEB1001X:RESC1005X40N, symbol Device:R
- added R65, R66, R67, R71, R72, R73, R74, R75, R76, R78: 10k, CMP2010-FX-1002ELF:RESC5025X70N, symbol Device:R
- added U1, U9: LM324A, LM324N:DIP794W56P254L1905H533Q14N, symbol Amplifier_Operational:LM324A
- J19: renamed from J?; footprint (none) -> Connector_PinHeader_1.00mm:PinHeader_1x05_P1.00mm_Vertical
Connections:
- net +12V is gone; now on net 5V: IC13.3 (+IN), U5.4 (V+), U7.4 (V+)
- net -12V is gone; now on net GND: IC13.4 (-IN), U5.11 (V-), U7.11 (V-)
- net 5V: now also R63.1, U1.4 (V+), U9.4 (V+)
- net GND: now also C41.2, R64.2, U1.11 (V-), U9.11 (V-)
- net at C1.2: now also R74.2, U1.14; no longer J6.3
- net at R3.1: now also R73.2, U1.8; no longer J4.2
- net at R9.1: now also R76.2, U9.7; no longer J5.3
- net at R4.1: now also R78.2, U9.8; no longer J5.2
- net at R8.1: now also R75.2, U1.7; no longer J4.3
- net at J6.2: now also J6.3, C55.1
- net SD_Step-Up: no longer names the net of IC10.19 (PB1)
- net SD_Step-Up: no longer J3.2 (Pin_2)
- new net: C44.1, J4.2
- new net: C56.1, J4.3
- new net: C41.1, R63.2, R64.1, U1.3 (+)
- new net: R71.2, R76.1, U9.6 (-)
- new net: R72.2, R78.1, U9.9 (-)
- new net: C57.1, J5.3
- new net: C57.2, R71.1
- new net: C58.2, R72.1
- new net: C58.1, J5.2
- new net: R65.2, R73.1, U1.9 (-)
- new net: R67.2, R75.1, U1.6 (-)
- new net: C56.2, R67.1
- new net: C44.2, R65.1
- new net: R66.2, R74.1, U1.13 (-)
- new net: C55.2, R66.1
- new net Vmp: U1.1, U1.10 (+), U1.12 (+), U1.2 (-), U1.5 (+), U9.10 (+), U9.5 (+)
Other:
- moved on the sheet: C36, C37, J4, J5, J6, PS1

Commit message: Word document aangepast
Parts:
- removed C55: 1µ, C0805X105K8RAC7210:CAPC2012X100N, symbol Device:C
- removed IC13: LMV321AUIDBVR, LMV321AUIDBVR:SOT95P280X145-5N, symbol LMV321AUIDBVR:LMV321AUIDBVR
- removed R66, R74: 10k, CMP2010-FX-1002ELF:RESC5025X70N, symbol Device:R
Connections:
- net POT1_A: now also U1.14
- net at R1.2, R2.1: now also U1.13 (-)
- net at C1.2: now also J6.2, J6.3; no longer U1.14
- no-connect marks 81 -> 82
Other:
- moved on the sheet: J6, U1D
Changed lines of the file:
@@
 	20820 4870 20960 4870
 Wire Wire Line
-	20520 4670 21460 4670
-Wire Wire Line
-	21460 4270 21460 4670
+	21470 4270 21470 4670
 $Comp
 L Device:CP C19
@@
 	20060 3570 20270 3570
 Wire Wire Line
-	21210 4270 21460 4270
-Wire Wire Line
 	20720 4270 20720 3570
 Wire Wire Line
@@
 L mengpaneel-rescue:SJ-63053A-SJ-63053A J6
 U 1 1 6D90AE19
-P 16880 3670
-F 0 "J6" H 17280 3935 50  0000 C CNN
-F 1 "SJ-63053A" H 17280 3844 50  0000 C CNN
-F 2 "SJ-63053A:SJ63053A" H 17530 3770 50  0001 L CNN
-F 3 "https://www.mouser.mx/datasheet/2/670/sj_63053a-1890674.pdf" H 17530 3670 50  0001 L CNN
-F 4 "Phone Connectors audio jack, 6.35 mm, horizontal, 3 conductor, through hole, 0 switches, w/ nut" H 17530 3570 50  0001 L CNN "Description"
-F 5 "12.8" H 17530 3470 50  0001 L CNN "Height"
-F 6 "490-SJ-63053A" H 17530 3370 50  0001 L CNN "Mouser Part Number"
-F 7 "https://www.mouser.co.uk/ProductDetail/CUI-Devices/SJ-63053A?qs=hWgE7mdIu5Q5ZZx8mXk5JQ%3D%3D" H 17530 3270 50  0001 L CNN "Mouser Price/Stock"
-F 8 "CUI Inc." H 17530 3170 50  0001 L CNN "Manufacturer_Name"
-F 9 "SJ-63053A" H 17530 3070 50  0001 L CNN "Manufacturer_Part_Number"
-	1    16880 3670
+P 18780 3570
+F 0 "J6" H 19180 3835 50  0000 C CNN
+F 1 "SJ-63053A" H 19180 3744 50  0000 C CNN
+F 2 "SJ-63053A:SJ63053A" H 19430 3670 50  0001 L CNN
+F 3 "https://www.mouser.mx/datasheet/2/670/sj_63053a-1890674.pdf" H 19430 3570 50  0001 L CNN
+F 4 "Phone Connectors audio jack, 6.35 mm, horizontal, 3 conductor, through hole, 0 switches, w/ nut" H 19430 3470 50  0001 L CNN "Description"
+F 5 "12.8" H 19430 3370 50  0001 L CNN "Height"
+F 6 "490-SJ-63053A" H 19430 3270 50  0001 L CNN "Mouser Part Number"
+F 7 "https://www.mouser.co.uk/ProductDetail/CUI-Devices/SJ-63053A?qs=hWgE7mdIu5Q5ZZx8mXk5JQ%3D%3D" H 19430 3170 50  0001 L CNN "Mouser Price/Stock"
+F 8 "CUI Inc." H 19430 3070 50  0001 L CNN "Manufacturer_Name"
+F 9 "SJ-63053A" H 19430 2970 50  0001 L CNN "Manufacturer_Part_Number"
+	1    18780 3570
 	1    0    0    1
 $EndComp
@@
 L power:GND #PWR0194
 U 1 1 6D90AE1F
-P 16880 3670
-F 0 "#PWR0194" H 16880 3420 50  0001 C CNN
-F 1 "GND" H 16885 3497 50  0000 C CNN
-F 2 "" H 16880 3670 50  0001 C CNN
-F 3 "" H 16880 3670 50  0001 C CNN
-	1    16880 3670
+P 18780 3570
+F 0 "#PWR0194" H 18780 3320 50  0001 C CNN
+F 1 "GND" H 18785 3397 50  0000 C CNN
+F 2 "" H 18780 3570 50  0001 C CNN
+F 3 "" H 18780 3570 50  0001 C CNN
+	1    18780 3570
 	-1   0    0    -1
 $EndComp
@@
 Connection ~ 26140 18220
 Connection ~ 20720 3570
-Wire Wire Line
-	20840 3470 20840 3130
-Wire Wire Line
-	20840 3130 22040 3130
-Wire Wire Line
-	22040 3130 22040 4270
-Wire Wire Line
-	22040 4270 21460 4270
-Connection ~ 21460 4270
 Wire Notes Line
 	10260 12640 10260 18730
@@
 Text GLabel 22520 3600 1    50   Input ~ 0
 5V
-Text GLabel 20840 3670 3    50   Input ~ 0
-5V
-Wire Wire Line
-	21840 3570 21900 3570
-$Comp
-L LMV321AUIDBVR:LMV321AUIDBVR IC13
-U 1 1 64D50D66
-P 20840 3470
-F 0 "IC13" H 21340 3735 50  0000 C CNN
-F 1 "LMV321AUIDBVR" H 21340 3644 50  0000 C CNN
-F 2 "LMV321AUIDBVR:SOT95P280X145-5N" H 21690 3570 50  0001 L CNN
-F 3 "https://www.ti.com/lit/gpn/LMV321A" H 21690 3470 50  0001 L CNN
-F 4 "Operational Amplifiers - Op Amps Single Low-Voltage, Cost-Optimized Rail-to-Rail Output Operational Amplifier 5-SOT-23 -40 to 125" H 21690 3370 50  0001 L CNN "Description"
-F 5 "1.45" H 21690 3270 50  0001 L CNN "Height"
-F 6 "595-LMV321AUIDBVR" H 21690 3170 50  0001 L CNN "Mouser Part Number"
-F 7 "https://www.mouser.co.uk/ProductDetail/Texas-Instruments/LMV321AUIDBVR/?qs=GBLSl2AkirulEcoP6K7rtg%3D%3D" H 21690 3070 50  0001 L CNN "Mouser Price/Stock"
-F 8 "Texas Instruments" H 21690 2970 50  0001 L CNN "Manufacturer_Name"
-F 9 "LMV321AUIDBVR" H 21690 2870 50  0001 L CNN "Manufacturer_Part_Number"
-	1    20840 3470
-	1    0    0    -1
-$EndComp
 Wire Wire Line
 	20720 3570 20840 3570
-Wire Wire Line
-	21840 3470 21900 3470
-Wire Wire Line
-	21900 3470 21900 3570
-$Comp
-L power:GND #PWR0104
-U 1 1 5FAA7B85
-P 21900 3570
-F 0 "#PWR0104" H 21900 3320 50  0001 C CNN
-F 1 "GND" H 21905 3397 50  0000 C CNN
-F 2 "" H 21900 3570 50  0001 C CNN
-F 3 "" H 21900 3570 50  0001 C CNN
-	1    21900 3570
-	-1   0    0    -1
-$EndComp
-Connection ~ 21900 3570
 Text GLabel 15550 12900 1    50   Input ~ 0
 5V
@@
 Wire Wire Line
 	17720 6070 17390 6070
-Wire Wire Line
-	19420 4090 19420 3570
-Wire Wire Line
-	19420 3570 19370 3570
-Text GLabel 18770 3470 0    50   Input ~ 0
+Text GLabel 20840 3370 0    50   Input ~ 0
 Vmp
 Wire Wire Line
-	18160 3670 18350 3670
-Wire Wire Line
-	19200 4090 19420 4090
+	19580 3570 19670 3570
 Wire Wire Line
-	18710 3670 18770 3670
-Connection ~ 18710 3670
+	19580 3470 19670 3470
 Wire Wire Line
-	18650 3670 18710 3670
+	19670 3470 19670 3570
+Connection ~ 19670 3570
 Wire Wire Line
-	18710 4090 18900 4090
-Wire Wire Line
-	18710 3670 18710 4090
-$Comp
-L Device:R R74
-U 1 1 6D09B198
-P 19050 4090
-F 0 "R74" V 19257 4090 50  0000 C CNN
-F 1 "10k" V 19166 4090 50  0000 C CNN
-F 2 "CMP2010-FX-1002ELF:RESC5025X70N" V 18980 4090 50  0001 C CNN
-F 3 "~" H 19050 4090 50  0001 C CNN
-	1    19050 4090
-	0    -1   -1   0
-$EndComp
-$Comp
-L Device:R R66
-U 1 1 6D09B19E
-P 18500 3670
-F 0 "R66" V 18707 3670 50  0000 C CNN
-F 1 "10k" V 18616 3670 50  0000 C CNN
-F 2 "CMP2010-FX-1002ELF:RESC5025X70N" V 18430 3670 50  0001 C CNN
-F 3 "~" H 18500 3670 50  0001 C CNN
-	1    18500 3670
-	0    -1   -1   0
-$EndComp
-$Comp
-L Device:C C55
-U 1 1 6D09B1A4
-P 18010 3670
-F 0 "C55" V 18262 3670 50  0000 C CNN
-F 1 "1µ" V 18171 3670 50  0000 C CNN
-F 2 "C0805X105K8RAC7210:CAPC2012X100N" H 18048 3520 50  0001 C CNN
-F 3 "~" H 18010 3670 50  0001 C CNN
-	1    18010 3670
-	0    -1   -1   0
-$EndComp
-Wire Wire Line
-	19420 3570 19760 3570
-Connection ~ 19420 3570
-Wire Wire Line
-	17680 3670 17770 3670
-Wire Wire Line
-	17680 3570 17770 3570
-Wire Wire Line
-	17770 3570 17770 3670
-Connection ~ 17770 3670
-Wire Wire Line
-	17770 3670 17860 3670
+	19670 3570 19760 3570
 $Comp
 L Amplifier_Operational:LM324A U1
 U 4 1 6D81755F
-P 19070 3570
-F 0 "U1" H 19070 3937 50  0000 C CNN
-F 1 "LM324A" H 19070 3846 50  0000 C CNN
-F 2 "LM324N:DIP794W56P254L1905H533Q14N" H 19020 3670 50  0001 C CNN
-F 3 "http://www.ti.com/lit/ds/symlink/lm2902-n.pdf" H 19120 3770 50  0001 C CNN
-	4    19070 3570
+P 21140 3470
+F 0 "U1" H 21140 3837 50  0000 C CNN
+F 1 "LM324A" H 21140 3746 50  0000 C CNN
+F 2 "LM324N:DIP794W56P254L1905H533Q14N" H 21090 3570 50  0001 C CNN
+F 3 "http://www.ti.com/lit/ds/symlink/lm2902-n.pdf" H 21190 3670 50  0001 C CNN
+	4    21140 3470
 	1    0    0    -1
 $EndComp
@@
 NoConn ~ 12280 13380
 NoConn ~ 15780 11080
+Wire Wire Line
+	21440 3470 21470 3470
+Wire Wire Line
+	21470 3470 21470 4270
+Wire Wire Line
+	21210 4270 21470 4270
+Connection ~ 21470 4270
+Wire Wire Line
+	20520 4670 21470 4670
+NoConn ~ 19660 9990
 $EndSCHEMATC
