File: PCB/mengpaneel.kicad_pcb (KiCad board)
At the start: 2 copper layers, 22 parts, among them U11 AD5290, U13 AD5290, U14 AD5290, U15 AD5290, U16 AD5290, U17 AD5290, U18 AD5290, U19 AD5290, U2 AD5290, U20 AD5290, U21 AD5290, U22 AD5290, U23 AD5290, U27 AD5290, U28 AD5290, U29 AD5290, U3 AD5290, U31 LM3480-3.3, U32 STM32F413RGTx, U4 AD5290, U6 AD5290, U8 AD5290

Commit message: PCB bijna af
Parts:
- removed U18, U19, U20, U21, U22, U23, U27, U28, U29: AD5290, Package_SO:MSOP-10_3x3mm_P0.5mm
- removed U31: LM3480-3.3, Package_TO_SOT_SMD:SOT-23
- removed U32: STM32F413RGTx, Package_QFP:LQFP-64_10x10mm_P0.5mm
- added C1: 2,2µ, MAL219299601E3:CAPAE1050X1050N, B.Cu at (336.2, 58.8)
- added C10: 2,2µ, EMF212B7225KGHT:CAPC2012X135N, B.Cu at (349.8, 100.8)
- added C11: 2,2µ, MAL219299601E3:CAPAE1050X1050N, B.Cu at (321.2, 92.0)
- added C12: 2,2µ, MAL219299601E3:CAPAE1050X1050N, B.Cu at (358.8, 72.5)
- added C13: 6,8n, C0805F682K1RACAUTO:CAPC2012X100N, B.Cu at (342.0, 105.2)
- added C14: 1,5n, C0402C152J3GACAUTO:CAPC1005X55N, B.Cu at (352.5, 103.0)
- added C15: 2,2µ, MAL219299601E3:CAPAE1050X1050N, B.Cu at (363.8, 105.0)
- added C16: 4,7µ, EEE-FK1K4R7V:CAPAE660X610N, B.Cu at (317.0, 117.0)
- added C17: 1µ, C0805X105K8RAC7210:CAPC2012X100N, B.Cu at (342.5, 113.2)
- added C18: 4,7µ, EEE-FK1K4R7V:CAPAE660X610N, B.Cu at (379.2, 130.8)
- added C19: 2,2µ, MAL219299601E3:CAPAE1050X1050N, B.Cu at (364.2, 58.8)
- added C2: 1µ, C0805X105K8RAC7210:CAPC2012X100N, B.Cu at (337.2, 77.5)
- added C20: 4,7µ, EEE-FK1K4R7V:CAPAE660X610N, B.Cu at (379.2, 100.8)
- added C21: 2,2µ, EMF212B7225KGHT:CAPC2012X135N, B.Cu at (316.5, 101.8)
- added C22: 2,2µ, EMF212B7225KGHT:CAPC2012X135N, B.Cu at (308.0, 106.8)
- added C23: 2,2µ, EMF212B7225KGHT:CAPC2012X135N, B.Cu at (305.0, 103.5)
- added C24: 2,2µ, EMF212B7225KGHT:CAPC2012X135N, B.Cu at (366.5, 85.0)
- added C25: 2,2µ, EMF212B7225KGHT:CAPC2012X135N, B.Cu at (386.0, 89.5)
- added C26: 2,2µ, EMF212B7225KGHT:CAPC2012X135N, B.Cu at (382.7, 85.2)
- added C27: 1,5n, C0402C152J3GACAUTO:CAPC1005X55N, B.Cu at (309.8, 107.2)
- added C28: 6,8n, C0805F682K1RACAUTO:CAPC2012X100N, B.Cu at (306.9, 109.8)
- added C29: 6,8n, C0805F682K1RACAUTO:CAPC2012X100N, B.Cu at (387.8, 99.0)
- added C3: 1µ, C0805X105K8RAC7210:CAPC2012X100N, B.Cu at (337.2, 75.5)
- added C30: 1,5n, C0402C152J3GACAUTO:CAPC1005X55N, B.Cu at (389.5, 89.5)
- added C31: 1,5n, C0402C152J3GACAUTO:CAPC1005X55N, B.Cu at (386.7, 121.5)
- added C32: 6,8n, C0805F682K1RACAUTO:CAPC2012X100N, B.Cu at (386.2, 116.8)
- added C33: 1µ, C0805X105K8RAC7210:CAPC2012X100N, B.Cu at (346.2, 119.0)
- added C34: 1µ, C0805X105K8RAC7210:CAPC2012X100N, B.Cu at (389.8, 111.8)
- added C35: 1µ, C0805X105K8RAC7210:CAPC2012X100N, B.Cu at (362.0, 122.2)
- added C36: 0.1µ, 06031C104K4Z2A:CAPC1608X90N, B.Cu at (378.0, 35.8)
- added C37: 0.1µ, 06031C104K4Z2A:CAPC1608X90N, B.Cu at (370.8, 35.7)
- added C38: 4.7µ, JMK212B7475KGHT:CAPC2114X145N, B.Cu at (377.2, 52.1)
- added C39: 2,2µ, MAL219299601E3:CAPAE1050X1050N, B.Cu at (352.5, 58.8)
- added C4: 1µ, C0805X105K8RAC7210:CAPC2012X100N, B.Cu at (338.5, 80.2)
- added C40: 4.7µ, JMK212B7475KGHT:CAPC2114X145N, B.Cu at (375.0, 51.0)
- added C41: 390p, C0603C391J1HACTU:CAPC1608X87N, B.Cu at (368.2, 43.8)
- added C42: 100n, C1206C100K5RACTU:CAPC3216X88N, B.Cu at (281.2, 212.5)
- added C43: 100n, C1206C100K5RACTU:CAPC3216X88N, B.Cu at (384.5, 49.2)
- added C44: 10p, C1206C100K5RACTU:CAPC3216X88N, B.Cu at (380.5, 53.0)
- added C45: 1µ, C0805X105K8RAC7210:CAPC2012X100N, B.Cu at (376.5, 30.2)
- added C46: 10µ, TMK212BC6106KG-T:CAPC2114X145N, B.Cu at (365.5, 27.8)
- added C47: 18p, C0402C180F5GACTU:CAPC1005X55N, B.Cu at (265.8, 198.2)
- added C48: 0.1µ, 06031C104K4Z2A:CAPC1608X90N, B.Cu at (265.0, 213.8)
- added C49: 0.1µ, 06031C104K4Z2A:CAPC1608X90N, B.Cu at (260.5, 212.0)
- added C5: 1µ, C0805X105K8RAC7210:CAPC2012X100N, B.Cu at (338.8, 72.0)
- added C50: 10µ, TMK212BC6106KG-T:CAPC2114X145N, B.Cu at (233.5, 209.0)
- added C59: 0,1µ, 06031C104K4Z2A:CAPC1608X90N, B.Cu at (236.8, 202.0)
- added C6: 2,2µ, MAL219299601E3:CAPAE1050X1050N, B.Cu at (333.0, 92.0)
- added C60: 0,1µ, 06031C104K4Z2A:CAPC1608X90N, B.Cu at (234.0, 212.0)
- added C63: 0,1µ, 06031C104K4Z2A:CAPC1608X90N, B.Cu at (239.0, 205.8)
- added C64: 18p, C0402C180F5GACTU:CAPC1005X55N, B.Cu at (268.0, 209.0)
- added C7: 1µ, C0805X105K8RAC7210:CAPC2012X100N, B.Cu at (353.5, 98.8)
- added C71: 22µ, C0805C226K7PACTU:CAPC2012X140N, B.Cu at (386.5, 46.2)
- added C72: 0,1µ, 06031C104K4Z2A:CAPC1608X90N, B.Cu at (383.0, 46.5)
- added C73: 0.1µ, 06031C104K4Z2A:CAPC1608X90N, B.Cu at (382.2, 43.8)
- added C8: 4,7µ, EEE-FK1K4R7V:CAPAE660X610N, B.Cu at (359.0, 131.2)
- added C9: 2,2µ, EMF212B7225KGHT:CAPC2012X135N, B.Cu at (346.5, 100.8)
- added D1: LED, 598-8C10-107F:LEDM2214X135N, F.Cu at (48.5, 37.2)
- added D10: LED, 598-8C80-107F:LEDM2214X135N, F.Cu at (48.5, 152.8)
- added D100: LED, 598-8C10-107F:LEDM2214X135N, F.Cu at (251.8, 75.8)
- added D101: LED, 598-8C30-107F:LEDM2214X135N, F.Cu at (251.8, 88.5)
- added D102: LED, 598-8C30-107F:LEDM2214X135N, F.Cu at (251.8, 101.2)
- added D103: LED, 598-8C30-107F:LEDM2214X135N, F.Cu at (251.8, 114.2)
- added D104: LED, 598-8C30-107F:LEDM2214X135N, F.Cu at (251.8, 127.0)
- added D105: LED, 598-8C80-107F:LEDM2214X135N, F.Cu at (251.8, 140.0)
- added D106: LED, 598-8C80-107F:LEDM2214X135N, F.Cu at (251.8, 152.8)
- added D107: LED, 598-8C80-107F:LEDM2214X135N, F.Cu at (251.8, 165.5)
- added D108: LED, 598-8C80-107F:LEDM2214X135N, F.Cu at (251.8, 178.2)
- added D109: LED, 598-8C10-107F:LEDM2214X135N, F.Cu at (276.8, 37.2)
- added D11: LED, 598-8C80-107F:LEDM2214X135N, F.Cu at (48.5, 165.5)
- added D110: LED, 598-8C10-107F:LEDM2214X135N, F.Cu at (276.8, 50.0)
- added D111: LED, 598-8C10-107F:LEDM2214X135N, F.Cu at (276.8, 62.8)
- added D112: LED, 598-8C10-107F:LEDM2214X135N, F.Cu at (276.8, 75.8)
- added D113: LED, 598-8C30-107F:LEDM2214X135N, F.Cu at (276.8, 88.5)
- added D114: LED, 598-8C30-107F:LEDM2214X135N, F.Cu at (276.8, 101.2)
- added D115: LED, 598-8C30-107F:LEDM2214X135N, F.Cu at (276.8, 114.2)
- added D116: LED, 598-8C30-107F:LEDM2214X135N, F.Cu at (276.8, 127.0)
- added D117: LED, 598-8C80-107F:LEDM2214X135N, F.Cu at (276.8, 140.0)
- added D118: LED, 598-8C80-107F:LEDM2214X135N, F.Cu at (276.8, 152.8)
- added D119: LED, 598-8C80-107F:LEDM2214X135N, F.Cu at (276.8, 165.5)
- added D12: LED, 598-8C80-107F:LEDM2214X135N, F.Cu at (48.5, 178.5)
- added D120: LED, 598-8C80-107F:LEDM2214X135N, F.Cu at (276.8, 178.2)
- added D121: LED, 598-8C10-107F:LEDM2214X135N, F.Cu at (184.8, 202.8)
- added D122: LED, 598-8C10-107F:LEDM2214X135N, F.Cu at (172.0, 202.8)
- added D123: LED, 598-8C10-107F:LEDM2214X135N, F.Cu at (159.2, 202.8)
- added D124: LED, 598-8C10-107F:LEDM2214X135N, F.Cu at (146.2, 202.8)
- added D125: LED, 598-8C30-107F:LEDM2214X135N, F.Cu at (133.5, 202.8)
- added D126: LED, 598-8C30-107F:LEDM2214X135N, F.Cu at (120.5, 202.8)
- added D127: LED, 598-8C30-107F:LEDM2214X135N, F.Cu at (107.8, 202.8)
- added D128: LED, 598-8C30-107F:LEDM2214X135N, F.Cu at (95.0, 202.8)
- added D129: LED, 598-8C80-107F:LEDM2214X135N, F.Cu at (82.2, 202.8)
- added D13: LED, 598-8C10-107F:LEDM2214X135N, F.Cu at (73.5, 37.2)
- added D130: LED, 598-8C80-107F:LEDM2214X135N, F.Cu at (69.2, 202.8)
- added D131: LED, 598-8C80-107F:LEDM2214X135N, F.Cu at (56.5, 202.8)
- added D132: LED, 598-8C80-107F:LEDM2214X135N, F.Cu at (43.5, 202.8)
- added D14: LED, 598-8C10-107F:LEDM2214X135N, F.Cu at (73.5, 50.0)
- added D15: LED, 598-8C10-107F:LEDM2214X135N, F.Cu at (73.5, 62.8)
- added D16: LED, 598-8C10-107F:LEDM2214X135N, F.Cu at (73.5, 75.8)
- added D17: LED, 598-8C30-107F:LEDM2214X135N, F.Cu at (73.5, 88.5)
- added D18: LED, 598-8C30-107F:LEDM2214X135N, F.Cu at (73.5, 101.5)
- added D19: LED, 598-8C30-107F:LEDM2214X135N, F.Cu at (73.5, 114.2)
- added D2: LED, 598-8C10-107F:LEDM2214X135N, F.Cu at (48.5, 50.0)
- added D20: LED, 598-8C30-107F:LEDM2214X135N, F.Cu at (73.5, 127.0)
- added D21: LED, 598-8C80-107F:LEDM2214X135N, F.Cu at (73.5, 140.0)
- added D22: LED, 598-8C80-107F:LEDM2214X135N, F.Cu at (73.5, 152.8)
- added D23: LED, 598-8C80-107F:LEDM2214X135N, F.Cu at (73.5, 165.5)
- added D24: LED, 598-8C80-107F:LEDM2214X135N, F.Cu at (73.5, 178.5)
- added D25: LED, 598-8C10-107F:LEDM2214X135N, F.Cu at (98.5, 37.2)
- added D26: LED, 598-8C10-107F:LEDM2214X135N, F.Cu at (98.5, 50.0)
- added D27: LED, 598-8C10-107F:LEDM2214X135N, F.Cu at (98.5, 62.8)
- added D28: LED, 598-8C10-107F:LEDM2214X135N, F.Cu at (98.5, 75.8)
- added D29: LED, 598-8C30-107F:LEDM2214X135N, F.Cu at (98.5, 88.5)
- added D3: LED, 598-8C10-107F:LEDM2214X135N, F.Cu at (48.5, 62.8)
- added D30: LED, 598-8C30-107F:LEDM2214X135N, F.Cu at (98.5, 101.5)
- added D31: LED, 598-8C30-107F:LEDM2214X135N, F.Cu at (98.5, 114.2)
- added D32: LED, 598-8C30-107F:LEDM2214X135N, F.Cu at (98.5, 127.0)
- added D33: LED, 598-8C80-107F:LEDM2214X135N, F.Cu at (98.5, 140.0)
- added D34: LED, 598-8C80-107F:LEDM2214X135N, F.Cu at (98.5, 152.8)
- added D35: LED, 598-8C80-107F:LEDM2214X135N, F.Cu at (98.5, 165.5)
- added D36: LED, 598-8C80-107F:LEDM2214X135N, F.Cu at (98.5, 178.5)
- added D37: LED, 598-8C10-107F:LEDM2214X135N, F.Cu at (123.5, 37.2)
- added D38: LED, 598-8C10-107F:LEDM2214X135N, F.Cu at (123.5, 50.0)
- added D39: LED, 598-8C10-107F:LEDM2214X135N, F.Cu at (123.5, 62.8)
- added D4: LED, 598-8C10-107F:LEDM2214X135N, F.Cu at (48.5, 75.8)
- added D40: LED, 598-8C10-107F:LEDM2214X135N, F.Cu at (123.5, 75.8)
- added D41: LED, 598-8C30-107F:LEDM2214X135N, F.Cu at (123.5, 88.5)
- added D42: LED, 598-8C30-107F:LEDM2214X135N, F.Cu at (123.5, 101.5)
- added D43: LED, 598-8C30-107F:LEDM2214X135N, F.Cu at (123.5, 114.2)
- added D44: LED, 598-8C30-107F:LEDM2214X135N, F.Cu at (123.5, 127.0)
- added D45: LED, 598-8C80-107F:LEDM2214X135N, F.Cu at (123.5, 140.0)
- added D46: LED, 598-8C80-107F:LEDM2214X135N, F.Cu at (123.5, 152.8)
- added D47: LED, 598-8C80-107F:LEDM2214X135N, F.Cu at (123.5, 165.5)
- added D48: LED, 598-8C80-107F:LEDM2214X135N, F.Cu at (123.5, 178.5)
- added D49: LED, 598-8C10-107F:LEDM2214X135N, F.Cu at (150.8, 37.2)
- added D5: LED, 598-8C30-107F:LEDM2214X135N, F.Cu at (48.5, 88.5)
- added D50: LED, 598-8C10-107F:LEDM2214X135N, F.Cu at (150.8, 50.0)
- added D51: LED, 598-8C10-107F:LEDM2214X135N, F.Cu at (150.8, 62.8)
- added D52: LED, 598-8C10-107F:LEDM2214X135N, F.Cu at (150.8, 75.8)
- added D53: LED, 598-8C30-107F:LEDM2214X135N, F.Cu at (150.8, 88.5)
- added D54: LED, 598-8C30-107F:LEDM2214X135N, F.Cu at (150.8, 101.5)
- added D55: LED, 598-8C30-107F:LEDM2214X135N, F.Cu at (150.8, 114.2)
- added D56: LED, 598-8C30-107F:LEDM2214X135N, F.Cu at (150.8, 127.0)
- added D57: LED, 598-8C80-107F:LEDM2214X135N, F.Cu at (150.8, 140.0)
- added D58: LED, 598-8C80-107F:LEDM2214X135N, F.Cu at (150.8, 152.8)
- added D59: LED, 598-8C80-107F:LEDM2214X135N, F.Cu at (150.8, 165.5)
- added D6: LED, 598-8C30-107F:LEDM2214X135N, F.Cu at (48.5, 101.5)
- added D60: LED, 598-8C80-107F:LEDM2214X135N, F.Cu at (150.8, 178.5)
- added D61: LED, 598-8C10-107F:LEDM2214X135N, F.Cu at (175.8, 37.2)
- added D62: LED, 598-8C10-107F:LEDM2214X135N, F.Cu at (175.8, 50.0)
- added D63: LED, 598-8C10-107F:LEDM2214X135N, F.Cu at (175.8, 62.8)
- added D64: LED, 598-8C10-107F:LEDM2214X135N, F.Cu at (175.8, 75.8)
- added D65: LED, 598-8C30-107F:LEDM2214X135N, F.Cu at (175.8, 88.5)
- added D66: LED, 598-8C30-107F:LEDM2214X135N, F.Cu at (175.8, 101.5)
- added D67: LED, 598-8C30-107F:LEDM2214X135N, F.Cu at (175.8, 114.2)
- added D68: LED, 598-8C30-107F:LEDM2214X135N, F.Cu at (175.8, 127.0)
- added D69: LED, 598-8C80-107F:LEDM2214X135N, F.Cu at (175.8, 140.0)
- added D7: LED, 598-8C30-107F:LEDM2214X135N, F.Cu at (48.5, 114.2)
- added D70: LED, 598-8C80-107F:LEDM2214X135N, F.Cu at (175.8, 152.8)
- added D71: LED, 598-8C80-107F:LEDM2214X135N, F.Cu at (175.8, 165.5)
- added D72: LED, 598-8C80-107F:LEDM2214X135N, F.Cu at (175.8, 178.5)
- added D73: LED, 598-8C10-107F:LEDM2214X135N, F.Cu at (200.8, 37.2)
- added D74: LED, 598-8C10-107F:LEDM2214X135N, F.Cu at (200.8, 50.0)
- added D75: LED, 598-8C10-107F:LEDM2214X135N, F.Cu at (200.8, 62.8)
- added D76: LED, 598-8C10-107F:LEDM2214X135N, F.Cu at (200.8, 75.8)
- added D77: LED, 598-8C30-107F:LEDM2214X135N, F.Cu at (200.8, 88.5)
- added D78: LED, 598-8C30-107F:LEDM2214X135N, F.Cu at (200.8, 101.2)
- added D79: LED, 598-8C30-107F:LEDM2214X135N, F.Cu at (200.8, 114.2)
- added D8: LED, 598-8C30-107F:LEDM2214X135N, F.Cu at (48.5, 127.0)
- added D80: LED, 598-8C30-107F:LEDM2214X135N, F.Cu at (200.8, 127.0)
- added D81: LED, 598-8C80-107F:LEDM2214X135N, F.Cu at (200.8, 140.0)
- added D82: LED, 598-8C80-107F:LEDM2214X135N, F.Cu at (200.8, 152.8)
- added D83: LED, 598-8C80-107F:LEDM2214X135N, F.Cu at (200.8, 165.5)
- added D84: LED, 598-8C80-107F:LEDM2214X135N, F.Cu at (200.8, 178.5)
- added D85: LED, 598-8C10-107F:LEDM2214X135N, F.Cu at (225.8, 37.2)
- added D86: LED, 598-8C10-107F:LEDM2214X135N, F.Cu at (225.8, 50.0)
- added D87: LED, 598-8C10-107F:LEDM2214X135N, F.Cu at (225.8, 62.8)
- added D88: LED, 598-8C10-107F:LEDM2214X135N, F.Cu at (225.8, 75.8)
- added D89: LED, 598-8C30-107F:LEDM2214X135N, F.Cu at (225.8, 88.5)
- added D9: LED, 598-8C80-107F:LEDM2214X135N, F.Cu at (48.5, 140.0)
- added D90: LED, 598-8C30-107F:LEDM2214X135N, F.Cu at (225.8, 101.2)
- added D91: LED, 598-8C30-107F:LEDM2214X135N, F.Cu at (225.8, 114.2)
- added D92: LED, 598-8C30-107F:LEDM2214X135N, F.Cu at (225.8, 127.0)
- added D93: LED, 598-8C80-107F:LEDM2214X135N, F.Cu at (225.8, 140.0)
- added D94: LED, 598-8C80-107F:LEDM2214X135N, F.Cu at (225.8, 152.8)
- added D95: LED, 598-8C80-107F:LEDM2214X135N, F.Cu at (225.8, 165.5)
- added D96: LED, 598-8C80-107F:LEDM2214X135N, F.Cu at (225.8, 178.5)
- added D97: LED, 598-8C10-107F:LEDM2214X135N, F.Cu at (251.8, 37.2)
- added D98: LED, 598-8C10-107F:LEDM2214X135N, F.Cu at (251.8, 50.0)
- added D99: LED, 598-8C10-107F:LEDM2214X135N, F.Cu at (251.8, 62.8)
- added IC1: MAX7219CNG+, MAX7219CNG+:DIP794W56P254L3054H457Q24N, B.Cu at (293.8, 111.0)
- added IC10: STM32F411CEU7, STM32F411CEU7:QFN50P700X700X65-49N-D, B.Cu at (263.0, 206.2)
- added IC11: AD5204BRUZ10-REEL7, AD5204BRUZ10-REEL7:SOP65P640X120-24N, B.Cu at (310.5, 99.5)
- added IC12: LTC3631EMS8E#TRPBF, LTC3631EMS8E#TRPBF:SOP65P490X110-9N, B.Cu at (370.7, 28.6)
- added IC13: LMV321AUIDBVR, LMV321AUIDBVR:SOT95P280X145-5N, B.Cu at (344.2, 67.5)
- added IC2: MAX7219CNG+, MAX7219CNG+:DIP794W56P254L3054H457Q24N, B.Cu at (294.0, 73.2)
- added IC3: MTCH6301-I_ML, MTCH6301-I_ML:QFN65P800X800X100-45N-D, B.Cu at (240.0, 211.5)
- added IC4: LTC3121EDE#PBF, LTC3121EDE#PBF:SON50P300X400X80-13N-D, B.Cu at (378.8, 48.0)
- added IC5: AD5204BRUZ10-REEL7, AD5204BRUZ10-REEL7:SOP65P640X120-24N, B.Cu at (343.8, 76.5)
- added IC6: AD5204BRUZ10-REEL7, AD5204BRUZ10-REEL7:SOP65P640X120-24N, B.Cu at (379.2, 91.0)
- added IC7: LM3480IM3-3.3_NOPB, LM3480IM3-3.3_NOPB:SOT95P237X112-3N, B.Cu at (374.5, 36.0)
- added IC8: AD5204BRUZ10-REEL7, AD5204BRUZ10-REEL7:SOP65P640X120-24N, B.Cu at (346.5, 94.2)
- added IC9: AD5204BRUZ10-REEL7, AD5204BRUZ10-REEL7:SOP65P640X120-24N, B.Cu at (354.8, 85.2)
- added J1: UJ2-MIBH-G-SMT-TR, UJ2-MIBH-G-SMT-TR:UJ2MIBHGSMTTR, B.Cu at (378.0, 18.8)
- added J2: Screw_Terminal_01x03, Connector_PinHeader_1.00mm:PinHeader_1x03_P1.00mm_Vertical, B.Cu at (243.5, 227.0)
- added J3: Screw_Terminal_01x14, Connector_PinHeader_1.00mm:PinHeader_1x14_P1.00mm_Vertical, B.Cu at (285.5, 227.0)
- added J4: SJ-63053A, SJ-63053A:SJ63053A, B.Cu at (293.0, 32.5)
- added J5: SJ-63053A, SJ-63053A:SJ63053A, B.Cu at (312.8, 32.5)
- added J6: SJ-63053A, SJ-63053A:SJ63053A, B.Cu at (332.2, 32.5)
- added J7: SJ-63053A, SJ-63053A:SJ63053A, B.Cu at (353.2, 32.5)
- added L1: 6.8µ, SRP0512-6R8K:SRP05126R8K, B.Cu at (385.2, 31.5)
- added L2: 100µ, LQM21DN101M70L:VARC2012X145N, B.Cu at (376.5, 27.8)
- added R1: 1k, ERA-2VEB1001X:RESC1005X40N, B.Cu at (336.8, 67.5)
- added R10: 10k, CMP2010-FX-1002ELF:RESC5025X70N, B.Cu at (341.5, 129.8)
- added R11: 100k, ERJ-UP3D1003V:RESC1608X55N, B.Cu at (325.0, 118.5)
- added R12: 22k, RCS120622K0JNEA:RESC3216X65N, B.Cu at (336.2, 83.0)
- added R13: 10k, CMP2010-FX-1002ELF:RESC5025X70N, B.Cu at (332.8, 123.8)
- added R14: 22k, RCS120622K0JNEA:RESC3216X65N, B.Cu at (341.5, 120.8)
- added R15: 10k, CMP2010-FX-1002ELF:RESC5025X70N, B.Cu at (340.0, 123.8)
- added R16: 22k, RCS120622K0JNEA:RESC3216X65N, B.Cu at (347.8, 70.8)
- added R17: 22k, RCS120622K0JNEA:RESC3216X65N, B.Cu at (356.5, 100.0)
- added R18: 10k, CMP2010-FX-1002ELF:RESC5025X70N, B.Cu at (324.0, 111.2)
- added R19: 9,53k, CR0805-FX-9531ELF:RESC2012X60N, B.Cu at (285.0, 111.0)
- added R2: 100k, ERJ-UP3D1003V:RESC1608X55N, B.Cu at (340.0, 69.5)
- added R20: 9,53k, CR0805-FX-9531ELF:RESC2012X60N, B.Cu at (302.5, 73.5)
- added R21: 10k, CMP2010-FX-1002ELF:RESC5025X70N, B.Cu at (344.8, 109.5)
- added R22: 22k, RCS120622K0JNEA:RESC3216X65N, B.Cu at (345.5, 104.8)
- added R23: 10k, CMP2010-FX-1002ELF:RESC5025X70N, B.Cu at (341.5, 101.5)
- added R24: 10k, CMP2010-FX-1002ELF:RESC5025X70N, B.Cu at (367.5, 124.5)
- added R25: 10k, CMP2010-FX-1002ELF:RESC5025X70N, B.Cu at (371.5, 104.2)
- added R26: 100k, ERJ-UP3D1003V:RESC1608X55N, B.Cu at (324.8, 105.8)
- added R27: 22k, RCS120622K0JNEA:RESC3216X65N, B.Cu at (349.2, 106.0)
- added R28: 100k, ERJ-UP3D1003V:RESC1608X55N, B.Cu at (370.5, 122.8)
- added R29: 100k, ERJ-UP3D1003V:RESC1608X55N, B.Cu at (372.0, 109.8)
- added R3: 100k, ERJ-UP3D1003V:RESC1608X55N, B.Cu at (296.4, 53.5)
- added R30: 10k, CMP2010-FX-1002ELF:RESC5025X70N, B.Cu at (322.2, 102.0)
- added R31: 22k, RCS120622K0JNEA:RESC3216X65N, B.Cu at (316.2, 105.8)
- added R32: 10k, CMP2010-FX-1002ELF:RESC5025X70N, B.Cu at (318.2, 109.8)
- added R33: 10k, CMP2010-FX-1002ELF:RESC5025X70N, B.Cu at (318.8, 123.8)
- added R34: 22k, RCS120622K0JNEA:RESC3216X65N, B.Cu at (389.5, 93.8)
- added R35: 10k, CMP2010-FX-1002ELF:RESC5025X70N, B.Cu at (386.5, 94.8)
- added R36: 10k, CMP2010-FX-1002ELF:RESC5025X70N, B.Cu at (371.5, 97.2)
- added R37: 22k, RCS120622K0JNEA:RESC3216X65N, B.Cu at (371.0, 92.5)
- added R38: 10k, CMP2010-FX-1002ELF:RESC5025X70N, B.Cu at (364.2, 90.5)
- added R39: 10k, CMP2010-FX-1002ELF:RESC5025X70N, B.Cu at (312.2, 108.0)
- added R4: 100k, ERJ-UP3D1003V:RESC1608X55N, B.Cu at (315.8, 53.8)
- added R40: 22k, RCS120622K0JNEA:RESC3216X65N, B.Cu at (309.2, 113.0)
- added R41: 10k, CMP2010-FX-1002ELF:RESC5025X70N, B.Cu at (325.8, 123.8)
- added R42: 10k, CMP2010-FX-1002ELF:RESC5025X70N, B.Cu at (387.8, 106.2)
- added R43: 22k, RCS120622K0JNEA:RESC3216X65N, B.Cu at (387.0, 101.5)
- added R44: 10k, CMP2010-FX-1002ELF:RESC5025X70N, B.Cu at (388.1, 86.0)
- added R45: 10k, CMP2010-FX-1002ELF:RESC5025X70N, B.Cu at (364.2, 95.5)
- added R46: 22k, RCS120622K0JNEA:RESC3216X65N, B.Cu at (387.0, 123.8)
- added R47: 10k, CMP2010-FX-1002ELF:RESC5025X70N, B.Cu at (363.8, 81.2)
- added R48: 22k, RCS120622K0JNEA:RESC3216X65N, B.Cu at (341.5, 117.0)
- added R49: 22k, RCS120622K0JNEA:RESC3216X65N, B.Cu at (387.2, 112.5)
- added R5: 100k, ERJ-UP3D1003V:RESC1608X55N, B.Cu at (332.8, 78.0)
- added R50: 22k, RCS120622K0JNEA:RESC3216X65N, B.Cu at (362.8, 84.2)
- added R51: 200, CMP2010AFX-2000ELF:RESC5025X70N, B.Cu at (347.2, 114.5)
- added R52: 200, CMP2010AFX-2000ELF:RESC5025X70N, B.Cu at (366.2, 114.2)
- added R53: 200, CMP2010AFX-2000ELF:RESC5025X70N, B.Cu at (351.8, 119.0)
- added R54: 200, CMP2010AFX-2000ELF:RESC5025X70N, B.Cu at (356.5, 123.0)
- added R55: 100, CMP2010AFX-1000ELF:RESC5025X70N, B.Cu at (352.2, 111.0)
- added R56: 100, CMP2010AFX-1000ELF:RESC5025X70N, B.Cu at (357.0, 116.0)
- added R58: 100K, ERJ-UP3D1003V:RESC1608X55N, B.Cu at (264.5, 200.2)
- added R59: 1M, ERJ-UP3D1004V:RESC1608X55N, B.Cu at (364.5, 30.8)
- added R6: 100k, ERJ-UP3D1003V:RESC1608X55N, B.Cu at (334.5, 78.0)
- added R60: 71,5k, ERJ-UP3F7152V:RESC1608X55N, B.Cu at (366.2, 30.8)
- added R68: 1k, ERA-2VEB1001X:RESC1005X40N, B.Cu at (236.8, 217.8)
- added R69: 1k, ERA-2VEB1001X:RESC1005X40N, B.Cu at (234.0, 215.3)
- added R7: 22k, RCS120622K0JNEA:RESC3216X65N, B.Cu at (333.0, 75.2)
- added R70: 1k, ERA-2VEB1001X:RESC1005X40N, B.Cu at (233.5, 207.0)
- added R77: 20k, RCC04022K20FKED:RESC1005X40N, B.Cu at (240.5, 203.8)
- added R8: 100k, ERJ-UP3D1003V:RESC1608X55N, B.Cu at (291.2, 53.5)
- added R85: 57.6k, CR0603-FX-5762ELF:RESC1608X55N, B.Cu at (372.2, 43.8)
- added R86: 210k, RQ73C2A210KBTDF:RESC2012X65N, B.Cu at (376.0, 42.2)
- added R87: 1.02M, CRCW06031M02FKEA:RESC1608X50N, B.Cu at (385.0, 42.5)
- added R88: 113k, CR0805-FX-1133ELF:RESC2012X60N, B.Cu at (379.2, 43.5)
- added R9: 100k, ERJ-UP3D1003V:RESC1608X55N, B.Cu at (310.8, 53.8)
- added SW1: SW_Push, PTS526_SK15_SMTR2_LFS:PTS526SK15SMTR2LFS, B.Cu at (280.8, 206.0)
- added SW2: SW_DPDT_x2, Connector_PinHeader_1.00mm:PinHeader_1x06_P1.00mm_Vertical, B.Cu at (268.0, 227.0)
- added SW3: SW_DPST_x2, Connector_PinHeader_1.00mm:PinHeader_1x04_P1.00mm_Vertical, B.Cu at (258.5, 227.0)
- added SW4: SW_DPST_x2, Connector_PinHeader_1.00mm:PinHeader_1x04_P1.00mm_Vertical, B.Cu at (251.0, 227.0)
- added U5: LM324N, LM324N:DIP794W56P254L1905H533Q14N, B.Cu at (333.0, 112.0)
- added U7: LM324N, LM324N:DIP794W56P254L1905H533Q14N, B.Cu at (379.2, 116.2)
- added Y1: 8MHz, ECS-80-18-4X-CKM:ECS80184XCKM, B.Cu at (272.0, 207.0)
- U11, U14, U15, U16, U17, U2, U3, U4, U6, U8: value AD5290 -> Touchpad_mp; footprint Package_SO:MSOP-10_3x3mm_P0.5mm -> schema_tp:touchpad_footprint_normaal
- U13: value AD5290 -> Touchpad_mp_LR; footprint Package_SO:MSOP-10_3x3mm_P0.5mm -> schema_tp:touchpad_footprint_LR
- moved U6 124.3 mm to (26.8, 39.2)
- moved U15 122.1 mm to (255.0, 39.2)
- moved U13 114.3 mm to (181.8, 204.5), turned to 270 degrees
- moved U3 113.1 mm to (230.0, 39.2)
- moved U8 104.0 mm to (51.8, 39.2)
- moved U11 86.1 mm to (76.8, 39.2)
- moved U14 76.8 mm to (204.0, 39.2)
- moved U17 71.0 mm to (101.8, 39.2)
- moved U2 67.9 mm to (179.0, 39.2)
- moved U4 59.5 mm to (129.0, 39.2)
- moved U16 45.0 mm to (154.0, 39.2)
Connections:
- U11 pad 1: Net-(C22-Pad1) -> slider_6
- U11 pad 10: Net-(C28-Pad1) -> Net-(U11-Pad10)
- U11 pad 2: Net-(C22-Pad2) -> Net-(U11-Pad2)
- U11 pad 3: -15V -> Net-(U11-Pad3)
- U11 pad 4: GND -> Net-(U11-Pad4)
- U11 pad 5: CS_POT -> Net-(U11-Pad5)
- U11 pad 6: CLK -> Net-(U11-Pad6)
- U11 pad 7: L1.7 -> Net-(U11-Pad7)
- U11 pad 9: +15V -> Net-(U11-Pad9)
- U13 pad 1: Net-(C21-Pad2) -> slider_7
- U13 pad 10: Net-(R48-Pad1) -> laag4_9
- U13 pad 2: Net-(C21-Pad1) -> laag4_1
- U13 pad 3: -15V -> laag4_2
- U13 pad 4: GND -> laag4_3
- U13 pad 5: CS_POT -> laag4_4
- U13 pad 6: CLK -> laag4_5
- U13 pad 7: Din2_POT -> laag4_6
- U13 pad 8: L2.1 -> laag4_7
- U13 pad 9: +15V -> laag4_8
- U14 pad 1: Net-(R30-Pad2) -> slider_9
- U14 pad 10: Net-(C27-Pad1) -> Net-(U14-Pad10)
- U14 pad 2: Net-(R39-Pad1) -> Net-(U14-Pad2)
- U14 pad 3: -15V -> Net-(U14-Pad3)
- U14 pad 4: GND -> Net-(U14-Pad4)
- U14 pad 5: CS_POT -> Net-(U14-Pad5)
- U14 pad 6: CLK -> Net-(U14-Pad6)
- U14 pad 7: L1.6 -> Net-(U14-Pad7)
- U14 pad 8: L1.7 -> Net-(U14-Pad8)
- U14 pad 9: +15V -> Net-(U14-Pad9)
- U15 pad 1: Net-(C10-Pad1) -> slider_10
- U15 pad 10: Net-(C13-Pad1) -> Net-(U15-Pad10)
- U15 pad 2: Net-(C10-Pad2) -> Net-(U15-Pad2)
- U15 pad 3: -15V -> Net-(U15-Pad3)
- U15 pad 4: GND -> Net-(U15-Pad4)
- U15 pad 5: CS_POT -> Net-(U15-Pad5)
- U15 pad 6: CLK -> Net-(U15-Pad6)
- U15 pad 7: L1.4 -> Net-(U15-Pad7)
- U15 pad 8: L1.5 -> Net-(U15-Pad8)
- U15 pad 9: +15V -> Net-(U15-Pad9)
- U16 pad 1: Net-(R13-Pad2) -> slider_8
- U16 pad 10: Net-(C14-Pad1) -> Net-(U16-Pad10)
- U16 pad 2: Net-(R23-Pad1) -> Net-(U16-Pad2)
- U16 pad 3: -15V -> Net-(U16-Pad3)
- U16 pad 4: GND -> Net-(U16-Pad4)
- U16 pad 5: CS_POT -> Net-(U16-Pad5)
- U16 pad 6: CLK -> Net-(U16-Pad6)
- U16 pad 7: L1.5 -> Net-(U16-Pad7)
- U16 pad 8: L1.6 -> Net-(U16-Pad8)
- U16 pad 9: +15V -> Net-(U16-Pad9)
- U17 pad 1: Net-(C9-Pad2) -> slider_11
- U17 pad 10: Net-(R27-Pad1) -> Net-(U11-Pad22)
- U17 pad 2: Net-(C9-Pad1) -> Net-(U11-Pad14)
- U17 pad 3: -15V -> Net-(U11-Pad15)
- U17 pad 4: GND -> Net-(U11-Pad16)
- U17 pad 5: CS_POT -> Net-(U11-Pad17)
- U17 pad 6: CLK -> Net-(U11-Pad18)
- U17 pad 7: L1.3 -> Net-(U11-Pad19)
- U17 pad 8: L1.4 -> Net-(U11-Pad20)
- U17 pad 9: +15V -> Net-(U11-Pad21)
- U2 pad 1: Net-(R8-Pad2) -> slider_4
- U2 pad 10: Net-(C4-Pad1) -> laag2_9
- U2 pad 2: GND -> laag2_1
- U2 pad 3: -15V -> laag2_2
- U2 pad 4: GND -> laag2_3
- U2 pad 5: CS_POT -> laag2_4
- U2 pad 6: CLK -> laag2_5
- U2 pad 7: L1.2 -> laag2_6
- U2 pad 8: L1.3 -> laag2_7
- U2 pad 9: +15V -> laag2_8
- U3 pad 1: Net-(R2-Pad2) -> slider_5
- U3 pad 10: Net-(C2-Pad1) -> laag3_9
- U3 pad 2: GND -> laag3_1
- U3 pad 3: -15V -> laag3_2
- U3 pad 4: GND -> laag3_3
- U3 pad 5: CS_POT -> laag3_4
- U3 pad 6: CLK -> laag3_5
- U3 pad 7: Din1_POT -> laag3_6
- U3 pad 8: L1.1 -> laag3_7
- U3 pad 9: +15V -> laag3_8
- U4 pad 10: Net-(C5-Pad1) -> laag1_9
- U4 pad 2: GND -> laag1_1
- U4 pad 3: -15V -> laag1_2
- U4 pad 4: GND -> laag1_3
- U4 pad 5: Net-(U4-Pad5) -> laag1_4
- U4 pad 6: Net-(U4-Pad6) -> laag1_5
- U4 pad 7: Net-(U4-Pad7) -> laag1_6
- U4 pad 8: Net-(U4-Pad8) -> laag1_7
- U4 pad 9: +15V -> laag1_8
- U6 pad 1: Net-(R9-Pad2) -> slider_1
- U6 pad 10: Net-(C7-Pad1) -> laag_9
- U6 pad 2: GND -> laag_1
- U6 pad 3: -15V -> laag_2
- U6 pad 4: GND -> laag_3
- U6 pad 5: Net-(U6-Pad5) -> laag_4
- U6 pad 6: Net-(U6-Pad6) -> laag_5
- U6 pad 7: Net-(U6-Pad7) -> laag_6
- U6 pad 8: Net-(U6-Pad8) -> laag_7
- U6 pad 9: +15V -> laag_8
- U8 pad 1: Net-(R3-Pad2) -> slider_2
- U8 pad 10: Net-(C3-Pad1) -> Net-(U6-Pad22)
- U8 pad 2: GND -> Net-(U6-Pad14)
- U8 pad 3: -15V -> Net-(U6-Pad15)
- U8 pad 4: GND -> Net-(U6-Pad16)
- U8 pad 5: CS_POT -> Net-(U6-Pad17)
- U8 pad 6: CLK -> Net-(U6-Pad18)
- U8 pad 7: L1.1 -> Net-(U6-Pad19)
- U8 pad 8: L1.2 -> Net-(U6-Pad20)
- U8 pad 9: +15V -> Net-(U6-Pad21)
Routing:
- net GND: track 0.00 -> 512.3 mm
- net LEDslider_10: track 0.00 -> 155.7 mm, vias 0 -> 1
- net LEDslider_1: track 0.00 -> 141.3 mm
- net LEDslider_2: track 0.00 -> 141.3 mm
- net LEDslider_8: track 0.00 -> 141.2 mm
- net LEDslider_7: track 0.00 -> 141.2 mm
- net LEDslider_6: track 0.00 -> 141.2 mm
- net LEDslider_5: track 0.00 -> 141.2 mm
- net LEDslider_4: track 0.00 -> 141.2 mm
- net LEDslider_3: track 0.00 -> 141.2 mm
- net LEDslider_9: track 0.00 -> 141.0 mm
- net 5V: track 0.00 -> 108.5 mm, vias 0 -> 2
- net LEDlaag_12: track 0.00 -> 69.5 mm, vias 0 -> 1
- net +12V: track 0.00 -> 68.1 mm
- net 3.3V: track 0.00 -> 62.2 mm
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Other:
- board text added: "LIN1"
- board text added: "LIN2"
- board text added: "MICROFOON"
- board text added: "Mengpaneel"
- board text added: "OUT"
- board text added: "Stijn Van den Bossche & Hannes Hugaert"

Commit message: Ho ho ho vrolijke Pasen iedereen.🐇🧺🥚 pcb bijna af
Parts:
- moved R56 21.6 mm to (354.6, 94.5), turned to 180 degrees
- moved D121 12.3 mm to (197.0, 203.2)
- moved D122 12.3 mm to (184.2, 203.2)
- moved D123 12.3 mm to (171.5, 203.2)
- moved D124 12.3 mm to (158.5, 203.2)
- moved D125 12.3 mm to (145.8, 203.2)
- moved D126 12.3 mm to (132.8, 203.2)
- moved D127 12.3 mm to (120.0, 203.2)
- moved D128 12.3 mm to (107.2, 203.2)
- moved D129 12.3 mm to (94.5, 203.2)
- moved D130 12.3 mm to (81.5, 203.2)
- moved D131 12.3 mm to (68.8, 203.2)
- moved D132 12.3 mm to (55.8, 203.2)
- moved U13 12.3 mm to (194.0, 205.0)
- moved C50 3.95 mm to (230.2, 206.8)
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Routing:
- net LEDslider_11: track 0.00 -> 380.3 mm
- net 3.3V: track 62.2 -> 371.5 mm, vias 0 -> 11
- net GND: track 512.3 -> 781.8 mm, vias 0 -> 15
- net SD_Step-Up: track 0.00 -> 252.1 mm, vias 0 -> 3
- net SPI1_MOSI: track 0.00 -> 223.0 mm, vias 0 -> 9
- net SPI1_SCK: track 0.00 -> 221.3 mm, vias 0 -> 10
- net LEDlaag_12: track 69.5 -> 273.7 mm, vias 1 -> 7
- net CS_POT4: track 0.00 -> 191.7 mm, vias 0 -> 3
- net CS_POT1: track 0.00 -> 186.1 mm, vias 0 -> 5
- net -12V: track 33.0 -> 206.1 mm, vias 3 -> 10
- net CS_POT5: track 0.00 -> 171.2 mm, vias 0 -> 3
- net CS_POT2: track 0.00 -> 165.6 mm, vias 0 -> 5
- net 5V: track 108.5 -> 272.7 mm, vias 2 -> 15
- net cs_leds: track 0.00 -> 150.7 mm, vias 0 -> 1
- net POT12_B: track 2.04 -> 143.2 mm, vias 0 -> 4
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
Commit message: PCB af alleen nog wachten op touchsliders
Parts:
- C72, C73: footprint 06031C104K4Z2A:CAPC1608X90N -> 0603YC104J4T4A:CAPC1608X90N
- moved D1 4.32 mm to (47.8, 33.0)
- moved D10 4.32 mm to (47.8, 148.5)
- moved D11 4.32 mm to (47.8, 161.2)
- moved D12 4.32 mm to (47.8, 174.2)
- moved D2 4.32 mm to (47.8, 45.8)
- moved D3 4.32 mm to (47.8, 58.5)
- moved D37 4.32 mm to (124.2, 33.0)
- moved D38 4.32 mm to (124.2, 45.8)
- moved D39 4.32 mm to (124.2, 58.5)
- moved D4 4.32 mm to (47.8, 71.5)
- moved D40 4.32 mm to (124.2, 71.5)
- moved D41 4.32 mm to (124.2, 84.2)
- moved D42 4.32 mm to (124.2, 97.2)
- moved D43 4.32 mm to (124.2, 110.0)
- moved D44 4.32 mm to (124.2, 122.8)
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Connections:
- D14 pad 2: Net-(D14-Pad2) -> LEDlaag_11
- D2 pad 2: Net-(D14-Pad2) -> LEDlaag_11
- D26 pad 2: Net-(D14-Pad2) -> LEDlaag_11
- D38 pad 2: Net-(D14-Pad2) -> LEDlaag_11
- U13 pad 10: laag4_9 -> Net-(U13-Pad10)
- U13 pad 11: laag4_10 -> Net-(U13-Pad11)
- U13 pad 12: laag4_11 -> Net-(U13-Pad12)
- U13 pad 13: laag4_12 -> Net-(U13-Pad13)
- U13 pad 14: Net-(U13-Pad14) -> laag_1
- U13 pad 15: Net-(U13-Pad15) -> laag_2
- U13 pad 16: Net-(U13-Pad16) -> laag_3
- U13 pad 17: Net-(U13-Pad17) -> laag_4
- U13 pad 18: Net-(U13-Pad18) -> laag_5
- U13 pad 19: Net-(U13-Pad19) -> laag_6
- U13 pad 2: laag4_1 -> Net-(U13-Pad2)
- U13 pad 20: Net-(U13-Pad20) -> laag_7
- U13 pad 21: Net-(U13-Pad21) -> laag_8
- U13 pad 22: Net-(U13-Pad22) -> laag_9
- U13 pad 23: Net-(U13-Pad23) -> laag_10
- U13 pad 24: Net-(U13-Pad24) -> laag_11
- U13 pad 25: Net-(U13-Pad25) -> laag_12
- U13 pad 3: laag4_2 -> Net-(U13-Pad3)
- U13 pad 4: laag4_3 -> Net-(U13-Pad4)
- U13 pad 5: laag4_4 -> Net-(U13-Pad5)
- U13 pad 6: laag4_5 -> Net-(U13-Pad6)
- U13 pad 7: laag4_6 -> Net-(U13-Pad7)
- U13 pad 8: laag4_7 -> Net-(U13-Pad8)
- U13 pad 9: laag4_8 -> Net-(U13-Pad9)
- U15 pad 14: laag4_1 -> Net-(U15-Pad14)
- U15 pad 15: laag4_2 -> Net-(U15-Pad15)
- U15 pad 16: laag4_3 -> Net-(U15-Pad16)
- U15 pad 17: laag4_4 -> Net-(U15-Pad17)
- U15 pad 18: laag4_5 -> Net-(U15-Pad18)
- U15 pad 19: laag4_6 -> Net-(U15-Pad19)
- U15 pad 20: laag4_7 -> Net-(U15-Pad20)
- U15 pad 21: laag4_8 -> Net-(U15-Pad21)
- U15 pad 22: laag4_9 -> Net-(U15-Pad22)
- U15 pad 23: laag4_10 -> Net-(U15-Pad23)
- U15 pad 24: laag4_11 -> Net-(U15-Pad24)
- U15 pad 25: laag4_12 -> Net-(U15-Pad25)
Routing:
- net LEDlaag_7: track 21.9 -> 1220.7 mm, vias 1 -> 23
- net LEDlaag_8: track 19.8 -> 1153.0 mm, vias 1 -> 25
- net LEDlaag_6: track 14.4 -> 1076.4 mm, vias 1 -> 21
- net LEDlaag_9: track 28.5 -> 1048.2 mm, vias 2 -> 24
- net LEDlaag_5: track 33.6 -> 953.9 mm, vias 1 -> 94
- net LEDlaag_10: track 22.0 -> 916.2 mm, vias 2 -> 43
- net LEDlaag_4: track 48.7 -> 840.2 mm, vias 1 -> 73
- net LEDlaag_11: track 38.7 -> 828.2 mm, vias 1 -> 41
- net LEDlaag_3: track 55.7 -> 721.7 mm, vias 2 -> 57
- net LEDlaag_2: track 59.2 -> 639.3 mm, vias 2 -> 39
- net LEDlaag_12: track 273.7 -> 755.5 mm, vias 7 -> 27
- net LEDlaag_1: track 68.7 -> 471.8 mm, vias 2 -> 21
- net LEDslider_1: track 141.3 -> 500.1 mm, vias 0 -> 4
- net LEDslider_2: track 141.3 -> 496.4 mm, vias 0 -> 8
- net LEDslider_3: track 141.2 -> 454.4 mm, vias 0 -> 7
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
Commit message: PCB af nu wachten op de docenten hun feedback.
Parts:
- moved U13 135.8 mm to (59.5, 223.8), turned to 90 degrees
- moved R58 2.31 mm to (263.4, 198.2)
- moved C49 1.00 mm to (260.5, 213.0)
- moved C63 0.50 mm to (235.8, 203.0)
Connections:
- IC10 pad 18: Net-(IC10-Pad18) -> GPIO_INT
- IC10 pad 19: Net-(IC10-Pad19) -> SD_Step-Up
- IC10 pad 20: Net-(IC10-Pad20) -> cs_leds
- IC10 pad 29: Net-(IC10-Pad29) -> UART_CLK
- IC10 pad 37: Net-(IC10-Pad37) -> CS_POT5
- IC10 pad 38: Net-(IC10-Pad38) -> CS_POT4
- IC10 pad 39: Net-(IC10-Pad39) -> CS_POT3
- IC10 pad 40: Net-(IC10-Pad40) -> CS_POT2
- IC10 pad 41: Net-(IC10-Pad41) -> CS_POT1
- SW2 pad 1: Net-(SW2-Pad1) -> Net-(IC10-Pad34)
- SW2 pad 3: Net-(SW2-Pad3) -> Net-(IC10-Pad33)
- SW3 pad 2: Net-(SW3-Pad2) -> Net-(IC10-Pad32)
- SW3 pad 4: Net-(SW3-Pad4) -> Net-(IC10-Pad27)
- SW4 pad 2: Net-(SW4-Pad2) -> Net-(IC10-Pad26)
- U13 pad 10: Net-(U13-Pad10) -> laag_9
- U13 pad 11: Net-(U13-Pad11) -> laag_10
- U13 pad 12: Net-(U13-Pad12) -> laag_11
- U13 pad 13: Net-(U13-Pad13) -> laag_12
- U13 pad 14: laag_1 -> Net-(U13-Pad14)
- U13 pad 15: laag_2 -> Net-(U13-Pad15)
- U13 pad 16: laag_3 -> Net-(U13-Pad16)
- U13 pad 17: laag_4 -> Net-(U13-Pad17)
- U13 pad 18: laag_5 -> Net-(U13-Pad18)
- U13 pad 19: laag_6 -> Net-(U13-Pad19)
- U13 pad 2: Net-(U13-Pad2) -> laag_1
- U13 pad 20: laag_7 -> Net-(U13-Pad20)
- U13 pad 21: laag_8 -> Net-(U13-Pad21)
- U13 pad 22: laag_9 -> Net-(U13-Pad22)
- U13 pad 23: laag_10 -> Net-(U13-Pad23)
- U13 pad 24: laag_11 -> Net-(U13-Pad24)
- U13 pad 25: laag_12 -> Net-(U13-Pad25)
- U13 pad 3: Net-(U13-Pad3) -> laag_2
- U13 pad 4: Net-(U13-Pad4) -> laag_3
- U13 pad 5: Net-(U13-Pad5) -> laag_4
- U13 pad 6: Net-(U13-Pad6) -> laag_5
- U13 pad 7: Net-(U13-Pad7) -> laag_6
- U13 pad 8: Net-(U13-Pad8) -> laag_7
- U13 pad 9: Net-(U13-Pad9) -> laag_8
- U4 pad 1: Net-(U4-Pad1) -> slider_3
Routing:
- net laag_12: track 0.00 -> 442.9 mm, vias 0 -> 7
- net laag_11: track 0.00 -> 424.4 mm, vias 0 -> 7
- net laag_10: track 0.00 -> 405.5 mm, vias 0 -> 7
- net laag_9: track 0.00 -> 395.3 mm, vias 0 -> 5
- net laag_8: track 0.00 -> 380.8 mm, vias 0 -> 5
- net laag_7: track 0.00 -> 366.4 mm, vias 0 -> 5
- net laag_6: track 0.00 -> 351.3 mm, vias 0 -> 5
- net laag_5: track 0.00 -> 340.3 mm, vias 0 -> 5
- net laag_4: track 0.00 -> 332.3 mm, vias 0 -> 5
- net laag_3: track 0.00 -> 319.4 mm, vias 0 -> 5
- net laag_2: track 0.00 -> 305.1 mm, vias 0 -> 5
- net laag_1: track 0.00 -> 289.7 mm, vias 0 -> 3
- net slider_1: track 0.00 -> 230.3 mm, vias 0 -> 4
- net slider_2: track 0.00 -> 210.1 mm, vias 0 -> 6
- net slider_6: track 0.00 -> 173.0 mm, vias 0 -> 4
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- added copper zone on B.Cu, net (none)
Other:
- board text added: "BASS"
- board text added: "MEDIUM"
- board text added: "MIC. VOLUME"
- board text added: "TREBLE"
- board text added: "VOLUME"
- board text added: "VOLUME OUT"

Commit message: edited PCB slightly to modify text for Bass - medium - treble
Other:
- board text added: "MASTER VOLUME"
- board text added: "MID"
- board text added: "TREB"
- board text added: "VOL"
- board text removed: "MEDIUM"
- board text removed: "TREBLE"
- board text removed: "VOLUME"
- board text removed: "VOLUME OUT"

Commit message: Kleine foutjes nog aangepast.
Parts:
- removed IC7: LM3480IM3-3.3_NOPB, LM3480IM3-3.3_NOPB:SOT95P237X112-3N
- added PS1: 173950336, 173950336:173950336, F.Cu at (375.5, 34.0)
- moved C37 7.27 mm to (363.5, 36.2), turned to 90 degrees
- moved C36 4.72 mm to (382.0, 38.2)
Routing:
- net GND: track 853.1 -> 859.8 mm
- net 5V: track 277.6 -> 282.3 mm, vias 15 -> 14
- net 3.3V: track 384.1 -> 382.5 mm
- removed copper zone on B.Cu, net (none)

Commit message: kleine aanpassing aan PCB
Parts:
- moved C45 1.50 mm to (376.5, 28.8)
- moved C46 1.50 mm to (365.5, 26.2)
- moved IC12 1.50 mm to (370.7, 27.1)
- moved L2 1.50 mm to (376.5, 26.2)
- moved R59 1.50 mm to (364.5, 29.2)
- moved R60 1.50 mm to (366.2, 29.2)
Routing:
- net -12V: track 208.6 -> 210.1 mm
- net 5V: track 282.3 -> 281.4 mm
