File: PCB/mengpaneel.kicad_pcb (KiCad board)
At the start: 2 copper layers, 296 parts, among them IC1 MAX7219CNG+, IC10 STM32F411CEU7, IC11 AD5204BRUZ10-REEL7, IC12 LTC3631EMS8E#TRPBF, IC13 LMV321AUIDBVR, IC2 MAX7219CNG+, IC3 MTCH6301-I_ML, IC4 LTC3121EDE#PBF, IC5 AD5204BRUZ10-REEL7, IC6 AD5204BRUZ10-REEL7, IC8 AD5204BRUZ10-REEL7, IC9 AD5204BRUZ10-REEL7, J1 UJ2-MIBH-G-SMT-TR, J2 Screw_Terminal_01x03, J3 Screw_Terminal_01x14, J4 SJ-63053A, J5 SJ-63053A, J6 SJ-63053A, J7 SJ-63053A, SW1 SW_Push, SW2 SW_DPDT_x2, SW3 SW_DPST_x2, SW4 SW_DPST_x2, U11 Touchpad_mp, U13 Touchpad_mp_LR, U14 Touchpad_mp, U15 Touchpad_mp, U16 Touchpad_mp, U17 Touchpad_mp, U2 Touchpad_mp, U3 Touchpad_mp, U4 Touchpad_mp, U5 LM324N, U6 Touchpad_mp, U7 LM324N, U8 Touchpad_mp, Y1 8MHz

Commit message: Document beginnen invullen
Parts:
- PS1: moved to B.Cu
- moved C1 11.3 mm to (342.8, 68.0)
- moved C10 11.3 mm to (356.2, 110.0)
- moved C11 11.3 mm to (327.8, 101.2)
- moved C12 11.3 mm to (365.2, 81.8)
- moved C13 11.3 mm to (348.5, 114.5)
- moved C14 11.3 mm to (359.0, 112.2)
- moved C15 11.3 mm to (370.2, 114.2)
- moved C16 11.3 mm to (323.5, 126.2)
- moved C17 11.3 mm to (349.0, 122.5)
- moved C18 11.3 mm to (385.8, 140.0)
- moved C19 11.3 mm to (370.8, 68.0)
- moved C2 11.3 mm to (343.7, 86.8)
- moved C20 11.3 mm to (385.8, 110.0)
- moved C21 11.3 mm to (323.0, 111.0)
- moved C22 11.3 mm to (314.5, 116.0)
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Routing:
- net -12V: track 210.1 -> 213.3 mm
- net GND: track 860.2 -> 862.7 mm
- net 3.3V: track 382.5 -> 383.7 mm

Commit message: PCB doet aan alle normen van de docent
Parts:
- removed C41: 390p, C0603C391J1HACTU:CAPC1608X87N
- removed C44: 10p, C1206C100K5RACTU:CAPC3216X88N
- removed C71: 22µ, C0805C226K7PACTU:CAPC2012X140N
- removed L1: 6.8µ, SRP0512-6R8K:SRP05126R8K
- removed R86: 210k, RQ73C2A210KBTDF:RESC2012X65N
- removed R87: 1.02M, CRCW06031M02FKEA:RESC1608X50N
- removed R88: 113k, CR0805-FX-1133ELF:RESC2012X60N
- added .: , Fuse:Fuse_0201_0603Metric, B.Cu at (244.2, 237.8)
- added ?: , Fuse:Fuse_0201_0603Metric, F.Cu at (235.2, 237.8)
- added ?: , Fuse:Fuse_0201_0603Metric, F.Cu at (238.2, 238.2)
- added ?: , Fuse:Fuse_0201_0603Metric, B.Cu at (223.5, 234.5)
- added ?: , Fuse:Fuse_0201_0603Metric, B.Cu at (220.8, 234.0)
- added ?: , Fuse:Fuse_0201_0603Metric, B.Cu at (233.5, 233.5)
- added ?: , Fuse:Fuse_0201_0603Metric, B.Cu at (246.2, 237.8)
- added ?: , Fuse:Fuse_0201_0603Metric, B.Cu at (232.5, 235.2)
- added C51: 4.7µ, JMK212B7475KGHT:CAPC2114X145N, B.Cu at (385.0, 47.5)
- added C52: 1n, C0402C102J4GACAUTO:CAPC1005X55N, B.Cu at (390.2, 67.8)
- added C53: 68p, 06035C680KAT2A:CAPC1608X90N, B.Cu at (385.2, 62.2)
- added C54: 47µ, C5750X7R1C476M230KB:CAPC5750X250N, B.Cu at (381.2, 71.5)
- added J10: Screw_Terminal_01x01, Connector_PinHeader_1.00mm:PinHeader_1x01_P1.00mm_Vertical, B.Cu at (151.0, 194.5)
- added J11: Screw_Terminal_01x01, Connector_PinHeader_1.00mm:PinHeader_1x01_P1.00mm_Vertical, B.Cu at (251.0, 208.8)
- added J12: Screw_Terminal_01x01, Connector_PinHeader_1.00mm:PinHeader_1x01_P1.00mm_Vertical, B.Cu at (213.2, 217.2)
- added J13: Screw_Terminal_01x01, Connector_PinHeader_1.00mm:PinHeader_1x01_P1.00mm_Vertical, B.Cu at (98.8, 194.5)
- added J14: Screw_Terminal_01x01, Connector_PinHeader_1.00mm:PinHeader_1x01_P1.00mm_Vertical, B.Cu at (218.0, 194.5)
- added J15: Screw_Terminal_01x01, Connector_PinHeader_1.00mm:PinHeader_1x01_P1.00mm_Vertical, B.Cu at (176.0, 194.5)
- added J16: Screw_Terminal_01x01, Connector_PinHeader_1.00mm:PinHeader_1x01_P1.00mm_Vertical, B.Cu at (254.8, 208.8)
- added J17: Screw_Terminal_01x01, Connector_PinHeader_1.00mm:PinHeader_1x01_P1.00mm_Vertical, B.Cu at (123.8, 194.5)
- added J18: Screw_Terminal_01x12, Connector_PinHeader_1.00mm:PinHeader_1x12_P1.00mm_Vertical, B.Cu at (246.2, 236.2)
- added J8: Screw_Terminal_01x01, Connector_PinHeader_1.00mm:PinHeader_1x01_P1.00mm_Vertical, B.Cu at (72.8, 194.5)
- added J9: Screw_Terminal_01x01, Connector_PinHeader_1.00mm:PinHeader_1x01_P1.00mm_Vertical, B.Cu at (201.0, 194.5)
- added L3: 3.3µ, SPM6530T-3R3M:INDPM7165X315N, B.Cu at (390.8, 40.5)
- added R57: 43.2k, CR0805-FX-4322ELF:RESC2012X60N, B.Cu at (388.0, 68.2)
- added R61: 383k, CR1206-FX-3833ELF:RESC3216X75N, B.Cu at (391.0, 51.2)
- added R62: 121k, CR0805-FX-1213ELF:RESC2012X60N, B.Cu at (384.5, 52.5)
- added SW2: SW_DPST_x2, Connector_PinHeader_1.00mm:PinHeader_1x04_P1.00mm_Vertical, B.Cu at (249.2, 236.2)
- added verbinding: , Fuse:Fuse_0201_0603Metric, B.Cu at (223.5, 232.8)
- added verbinding: , Fuse:Fuse_0201_0603Metric, B.Cu at (174.0, 194.2)
- added verbinding: , Fuse:Fuse_0201_0603Metric, B.Cu at (149.0, 194.2)
- added verbinding: , Fuse:Fuse_0201_0603Metric, B.Cu at (121.8, 194.2)
- added verbinding: , Fuse:Fuse_0201_0603Metric, B.Cu at (96.8, 194.2)
- added verbinding: , Fuse:Fuse_0201_0603Metric, B.Cu at (70.8, 194.2)
- added verbinding: , Fuse:Fuse_0201_0603Metric, B.Cu at (45.2, 194.2)
- added verbinding: , Fuse:Fuse_0201_0603Metric, B.Cu at (235.2, 232.2)
- added verbinding: , Fuse:Fuse_0201_0603Metric, F.Cu at (240.8, 239.0)
- added verbinding: , Fuse:Fuse_0201_0603Metric, B.Cu at (245.2, 237.8)
- added verbinding: , Fuse:Fuse_0201_0603Metric, B.Cu at (213.2, 219.0)
- added verbinding: , Fuse:Fuse_0201_0603Metric, B.Cu at (256.7, 208.8)
- added verbinding: , Fuse:Fuse_0201_0603Metric, B.Cu at (251.0, 207.5)
- added verbinding: , Fuse:Fuse_0201_0603Metric, B.Cu at (221.0, 194.0)
- added verbinding: , Fuse:Fuse_0201_0603Metric, B.Cu at (199.0, 194.2)
- C72: value 0,1µ -> 0.1µ
- J2: value Screw_Terminal_01x03 -> Screw_Terminal_01x01; footprint Connector_PinHeader_1.00mm:PinHeader_1x03_P1.00mm_Vertical -> Connector_PinHeader_1.00mm:PinHeader_1x01_P1.00mm_Vertical
- moved J2 207.0 mm to (47.2, 194.5), turned to 0 degrees
- moved SW4 2.25 mm to (255.2, 236.2), turned to 270 degrees
- moved C1 1.25 mm to (341.5, 68.0)
- moved C10 1.25 mm to (355.0, 110.0)
- moved C11 1.25 mm to (326.5, 101.2)
- moved C12 1.25 mm to (364.0, 81.8)
- moved C13 1.25 mm to (347.2, 114.5)
- moved C14 1.25 mm to (357.8, 112.2)
- moved C15 1.25 mm to (369.0, 114.2)
- moved C16 1.25 mm to (322.2, 126.2)
- moved C17 1.25 mm to (347.8, 122.5)
- moved C18 1.25 mm to (384.5, 140.0)
- moved C19 1.25 mm to (369.5, 68.0)
- moved C2 1.25 mm to (342.4, 86.8)
- moved C20 1.25 mm to (384.5, 110.0)
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Connections:
- IC10 pad 29: UART_CLK -> Net-(IC10-Pad29)
- IC10 pad 30: TX_UART -> Net-(IC10-Pad30)
- IC10 pad 31: RX_UART -> ID
- IC10 pad 32: Net-(IC10-Pad32) -> Data-
- IC10 pad 33: Net-(IC10-Pad33) -> Data+
- IC4 pad 4: GND -> Net-(C40-Pad1)
- J1 pad 2: Net-(J1-Pad2) -> Data-
- J1 pad 3: Net-(J1-Pad3) -> Data+
- J1 pad 4: Net-(J1-Pad4) -> ID
- J2 pad 1: RX_UART -> slider_1
- SW2 pad 4: (no net) -> Data+
- SW2 pad 5: (no net) -> ID
- SW2 pad 6: (no net) -> Data-
- SW3 pad 2: Net-(IC10-Pad32) -> Net-(IC10-Pad29)
Routing:
- net Data+: track 0.00 -> 377.2 mm, vias 0 -> 5
- net Data-: track 0.00 -> 373.6 mm, vias 0 -> 4
- net ID: track 0.00 -> 373.1 mm, vias 0 -> 4
- net laag_2: track 305.1 -> 334.9 mm
- net UART_CLK: track 29.4 -> 0.00 mm, vias 1 -> 0
- net laag_12: track 442.9 -> 472.2 mm
- net laag_3: track 319.4 -> 348.6 mm
- net Net-(IC10-Pad32): track 28.9 -> 0.00 mm, vias 5 -> 0
- net Net-(IC10-Pad30): track 0.00 -> 28.9 mm, vias 0 -> 1
- net TX_UART: track 28.7 -> 0.00 mm
- net RX_UART: track 28.6 -> 0.00 mm, vias 2 -> 0
- net laag_4: track 332.3 -> 360.1 mm
- net Net-(IC10-Pad33): track 27.7 -> 0.00 mm, vias 3 -> 0
- net laag_5: track 340.3 -> 367.5 mm, vias 5 -> 4
- net laag_11: track 424.4 -> 449.8 mm
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Other:
- board text added: "14 13 12 11 10 9 8 7 6 5 4 3 2 1"
- board text added: "2 1"
- board text added: "3 2 1"
- board text added: "5 4 3 2 1"

Commit message: Document bij getypt.
Parts:
- renumbered SW2 to SW_Extra
Changed lines of the file:
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@@
     (descr "Through hole straight pin header, 1x06, 1.00mm pitch, single row")
     (tags "Through hole pin header THT 1x06 1.00mm single row")
-    (fp_text reference SW2 (at 0 1.56 270) (layer B.SilkS)
+    (fp_text reference SW_Extra (at 0 1.56 270) (layer B.SilkS)
       (effects (font (size 1 1) (thickness 0.15)) (justify mirror))
     )
@@
   (segment (start 260.75 209) (end 260.75 209) (width 0.25) (layer F.Cu) (net 159))
   (via (at 260.75 209) (size 0.8) (drill 0.4) (layers F.Cu B.Cu) (net 159))
-  (via (at 258.75 217) (size 0.8) (drill 0.4) (layers F.Cu B.Cu) (net 159))
   (segment (start 259.473001 217.399999) (end 261.75 219.676998) (width 0.25) (layer F.Cu) (net 159))
   (segment (start 258.75 217) (end 259.149999 217.399999) (width 0.25) (layer F.Cu) (net 159))
@@
   (segment (start 267.75 230.25) (end 266.75 230.25) (width 0.25) (layer B.Cu) (net 159))
   (segment (start 269.5 232) (end 267.75 230.25) (width 0.25) (layer B.Cu) (net 159))
+  (via (at 258.75 217) (size 0.8) (drill 0.4) (layers F.Cu B.Cu) (net 159) (status 1000000))
   (segment (start 252.25 223.5) (end 252.25 223.75) (width 0.25) (layer B.Cu) (net 160))
   (segment (start 252.25 225.27282) (end 249.77282 227.75) (width 0.25) (layer B.Cu) (net 160))
@@
   (segment (start 263.75 213.5) (end 263.75 213.5) (width 0.25) (layer B.Cu) (net 161))
   (via (at 263.75 213.5) (size 0.8) (drill 0.4) (layers F.Cu B.Cu) (net 161))
-  (segment (start 263.75 213.5) (end 263.75 218.75) (width 0.25) (layer F.Cu) (net 161))
   (segment (start 263.75 218.84077) (end 264.5 219.59077) (width 0.25) (layer F.Cu) (net 161))
   (segment (start 263.75 218.75) (end 263.75 218.84077) (width 0.25) (layer F.Cu) (net 161))
@@
   (segment (start 270.25 231.75) (end 270.25 232) (width 0.25) (layer B.Cu) (net 161))
   (segment (start 270.25 232) (end 270.25 232) (width 0.25) (layer B.Cu) (net 161))
+  (segment (start 269 226.5) (end 266 223.5) (width 0.25) (layer F.Cu) (net 161))
+  (segment (start 269 230.25) (end 269 226.5) (width 0.25) (layer F.Cu) (net 161))
+  (segment (start 263.75 213.5) (end 263.75 218.75) (width 0.25) (layer F.Cu) (net 161))
   (via (at 270.25 232) (size 0.8) (drill 0.4) (layers F.Cu B.Cu) (net 161))
-  (segment (start 270.25 233.073002) (end 271.676998 234.5) (width 0.25) (layer F.Cu) (net 161))
   (segment (start 270.25 232) (end 270.25 233.073002) (width 0.25) (layer F.Cu) (net 161))
+  (segment (start 270.25 233.073002) (end 271.676998 234.5) (width 0.25) (layer F.Cu) (net 161))
+  (segment (start 271.676998 234.5) (end 272.175 234.5) (width 0.25) (layer F.Cu) (net 161))
   (segment (start 273.25 235.575) (end 273.25 236.25) (width 0.25) (layer F.Cu) (net 161))
   (segment (start 272.175 234.5) (end 273.25 235.575) (width 0.25) (layer F.Cu) (net 161))
-  (segment (start 271.676998 234.5) (end 272.175 234.5) (width 0.25) (layer F.Cu) (net 161))
-  (segment (start 269 226.5) (end 266 223.5) (width 0.25) (layer F.Cu) (net 161))
-  (segment (start 269 230.25) (end 269 226.5) (width 0.25) (layer F.Cu) (net 161))
   (segment (start 264.8 214.25) (end 264.75 214.25) (width 0.25) (layer B.Cu) (net 378))
   (via (at 262.75 232) (size 0.8) (drill 0.4) (layers F.Cu B.Cu) (net 382))
@@
   (segment (start 263.50437 215.82499) (end 263.913601 215.824989) (width 0.25) (layer B.Cu) (net 381))
   (segment (start 257.75 229.25) (end 257.75 221.86359) (width 0.25) (layer B.Cu) (net 381))
-  (segment (start 257.75 221.86359) (end 261.349982 218.263608) (width 0.25) (layer B.Cu) (net 381))
-  (segment (start 261.349982 218.263608) (end 261.349982 217.979379) (width 0.25) (layer B.Cu) (net 381))
   (segment (start 261.349982 217.979379) (end 263.50437 215.82499) (width 0.25) (layer B.Cu) (net 381))
+  (segment (start 261.349982 218.263608) (end 261.349982 217.979379) (width 0.25) (layer B.Cu) (net 381))
+  (segment (start 257.75 221.86359) (end 261.349982 218.263608) (width 0.25) (layer B.Cu) (net 381))
   (segment (start 264.114999 216.260001) (end 264.125 216.25) (width 0.25) (layer B.Cu) (net 382))
   (segment (start 264.114999 216.274999) (end 264.114999 216.260001) (width 0.25) (layer B.Cu) (net 382))

Commit message: word in git steken.
Connections:
- C45 pad 1: 5V -> +12V
- IC12 pad 2: 5V -> +12V
- IC12 pad 5: 5V -> +12V
Routing:
- net +12V: track 187.4 -> 225.9 mm, vias 6 -> 8
- net 5V: track 282.3 -> 276.8 mm, vias 14 -> 16

Commit message: pcb oke
Parts:
- removed C38, C40, C51: 4.7µ, JMK212B7475KGHT:CAPC2114X145N
- removed C43: 100n, C1206C100K5RACTU:CAPC3216X88N
- removed C45: 1µ, C0805X105K8RAC7210:CAPC2012X100N
- removed C46: 10µ, TMK212BC6106KG-T:CAPC2114X145N
- removed C52: 1n, C0402C102J4GACAUTO:CAPC1005X55N
- removed C53: 68p, 06035C680KAT2A:CAPC1608X90N
- removed C54: 47µ, C5750X7R1C476M230KB:CAPC5750X250N
- removed C72, C73: 0.1µ, 0603YC104J4T4A:CAPC1608X90N
- removed IC12: LTC3631EMS8E#TRPBF, LTC3631EMS8E#TRPBF:SOP65P490X110-9N
- removed IC4: LTC3121EDE#PBF, LTC3121EDE#PBF:SON50P300X400X80-13N-D
- removed L2: 100µ, LQM21DN101M70L:VARC2012X145N
- removed L3: 3.3µ, SPM6530T-3R3M:INDPM7165X315N
- removed R57: 43.2k, CR0805-FX-4322ELF:RESC2012X60N
- removed R59: 1M, ERJ-UP3D1004V:RESC1608X55N
- removed R60: 71,5k, ERJ-UP3F7152V:RESC1608X55N
- removed R61: 383k, CR1206-FX-3833ELF:RESC3216X75N
- removed R62: 121k, CR0805-FX-1213ELF:RESC2012X60N
- removed R85: 57.6k, CR0603-FX-5762ELF:RESC1608X55N
- removed SW_Extra: SW_DPDT_x2, Connector_PinHeader_1.00mm:PinHeader_1x06_P1.00mm_Vertical
- added C41: 0.1µ, 06031C104K4Z2A:CAPC1608X90N, B.Cu at (378.9, 58.2)
- added C44: 1µ, C0805X105K8RAC7210:CAPC2012X100N, B.Cu at (301.3, 57.5)
- added C55: 1µ, C0805X105K8RAC7210:CAPC2012X100N, B.Cu at (335.8, 59.5)
- added C56: 1µ, C0805X105K8RAC7210:CAPC2012X100N, B.Cu at (296.8, 59.0)
- added C57: 1µ, C0805X105K8RAC7210:CAPC2012X100N, B.Cu at (316.2, 59.2)
- added C58: 1µ, C0805X105K8RAC7210:CAPC2012X100N, B.Cu at (321.2, 57.5)
- added J19: Screw_Terminal_01x05, Connector_PinHeader_1.00mm:PinHeader_1x05_P1.00mm_Vertical, B.Cu at (272.8, 236.2)
- added R63: 1k, ERA-2VEB1001X:RESC1005X40N, B.Cu at (379.0, 63.0)
- added R64: 1k, ERA-2VEB1001X:RESC1005X40N, B.Cu at (378.8, 55.0)
- added R65: 10k, CMP2010-FX-1002ELF:RESC5025X70N, B.Cu at (396.8, 83.0)
- added R66: 10k, CMP2010-FX-1002ELF:RESC5025X70N, B.Cu at (396.8, 58.8)
- added R67: 10k, CMP2010-FX-1002ELF:RESC5025X70N, B.Cu at (379.2, 52.2)
- added R71: 10k, CMP2010-FX-1002ELF:RESC5025X70N, B.Cu at (379.2, 71.8)
- added R72: 10k, CMP2010-FX-1002ELF:RESC5025X70N, B.Cu at (378.2, 76.0)
- added R73: 10k, CMP2010-FX-1002ELF:RESC5025X70N, B.Cu at (396.8, 49.2)
- added R74: 10k, CMP2010-FX-1002ELF:RESC5025X70N, B.Cu at (396.8, 66.5)
- added R75: 10k, CMP2010-FX-1002ELF:RESC5025X70N, B.Cu at (307.8, 47.3)
- added R76: 10k, CMP2010-FX-1002ELF:RESC5025X70N, B.Cu at (380.8, 66.2)
- added R78: 10k, CMP2010-FX-1002ELF:RESC5025X70N, B.Cu at (396.8, 74.5)
- added U1: LM324A, LM324N:DIP794W56P254L1905H533Q14N, B.Cu at (388.0, 55.5)
- added U9: LM324A, LM324N:DIP794W56P254L1905H533Q14N, B.Cu at (388.0, 77.0)
- moved C36 9.19 mm to (380.8, 41.0), turned to 180 degrees
- moved C37 8.53 mm to (376.0, 41.0), turned to 0 degrees
- moved PS1 6.52 mm to (380.3, 36.8)
Connections:
- IC10 pad 19: SD_Step-Up -> Net-(IC10-Pad19)
- IC10 pad 31: ID -> Net-(IC10-Pad31)
- IC10 pad 32: Data- -> Net-(IC10-Pad32)
- IC10 pad 33: Data+ -> CS_POT5
- IC10 pad 34: Net-(IC10-Pad34) -> SWDIO
- IC10 pad 37: CS_POT5 -> SWCLK
- IC13 pad 3: +12V -> 5V
- IC13 pad 4: -12V -> GND
- J1 pad 2: Data- -> Net-(J1-Pad2)
- J1 pad 3: Data+ -> Net-(J1-Pad3)
- J1 pad 4: ID -> Net-(J1-Pad4)
- J3 pad 2: SD_Step-Up -> Net-(J3-Pad2)
- J4 pad 2: Net-(J4-Pad2) -> Net-(C44-Pad1)
- J4 pad 3: Net-(J4-Pad3) -> Net-(C56-Pad1)
- J5 pad 2: Net-(J5-Pad2) -> Net-(C58-Pad1)
- J5 pad 3: Net-(J5-Pad3) -> Net-(C57-Pad1)
- J6 pad 2: Net-(J6-Pad2) -> Net-(C55-Pad1)
- J6 pad 3: Net-(C1-Pad2) -> Net-(C55-Pad1)
- R3 pad 1: Net-(J4-Pad2) -> Net-(R3-Pad1)
- R4 pad 1: Net-(J5-Pad2) -> Net-(R4-Pad1)
- R8 pad 1: Net-(J4-Pad3) -> Net-(R75-Pad2)
- R9 pad 1: Net-(J5-Pad3) -> Net-(R76-Pad2)
- U5 pad 11: -12V -> GND
- U5 pad 4: +12V -> 5V
- U7 pad 11: -12V -> GND
- U7 pad 4: +12V -> 5V
Routing:
- net Data+: track 377.2 -> 0.00 mm, vias 5 -> 0
- net Data-: track 373.6 -> 0.00 mm, vias 4 -> 0
- net ID: track 373.1 -> 0.00 mm, vias 4 -> 0
- net SD_Step-Up: track 311.9 -> 0.00 mm, vias 8 -> 0
- net +12V: track 225.9 -> 0.00 mm, vias 8 -> 0
- net -12V: track 213.3 -> 0.00 mm, vias 10 -> 0
- net 5V: track 276.8 -> 401.7 mm, vias 16 -> 20
- net Net-(R3-Pad1): track 0.00 -> 115.1 mm
- net Net-(C44-Pad2): track 0.00 -> 112.0 mm, vias 0 -> 8
- net Net-(R75-Pad2): track 0.00 -> 104.0 mm, vias 0 -> 2
- net GND: track 882.6 -> 977.1 mm, vias 22 -> 29
- net Net-(C56-Pad2): track 0.00 -> 86.6 mm, vias 0 -> 4
- net Net-(R76-Pad2): track 0.00 -> 84.9 mm, vias 0 -> 6
- net Net-(R4-Pad1): track 0.00 -> 81.8 mm, vias 0 -> 5
- net Net-(R67-Pad2): track 0.00 -> 80.3 mm
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
Commit message: Word document aangepast
Parts:
- removed C55: 1µ, C0805X105K8RAC7210:CAPC2012X100N
- removed IC13: LMV321AUIDBVR, LMV321AUIDBVR:SOT95P280X145-5N
- removed R66, R74: 10k, CMP2010-FX-1002ELF:RESC5025X70N
- added REF**: MountingHole_3.2mm_M3_Pad_Via, MountingHole:MountingHole_3.2mm_M3_Pad_Via, F.Cu at (23.5, 237.8)
- added REF**: MountingHole_3.2mm_M3_Pad_Via, MountingHole:MountingHole_3.2mm_M3_Pad_Via, F.Cu at (23.5, 25.0)
- added REF**: MountingHole_3.2mm_M3_Pad_Via, MountingHole:MountingHole_3.2mm_M3_Pad_Via, F.Cu at (396.2, 237.8)
- added REF**: MountingHole_3.2mm_M3_Pad_Via, MountingHole:MountingHole_3.2mm_M3_Pad_Via, F.Cu at (396.2, 25.0)
Connections:
- J6 pad 2: Net-(C55-Pad1) -> Net-(C1-Pad2)
- J6 pad 3: Net-(C55-Pad1) -> Net-(C1-Pad2)
- R1 pad 2: Net-(IC13-Pad2) -> Net-(R1-Pad2)
- R2 pad 1: Net-(IC13-Pad2) -> Net-(R1-Pad2)
- U1 pad 13: Net-(R66-Pad2) -> Net-(R1-Pad2)
- U1 pad 14: Net-(C1-Pad2) -> POT1_A
Routing:
- net Net-(R1-Pad2): track 0.00 -> 76.0 mm, vias 0 -> 4
- net POT1_A: track 16.4 -> 85.1 mm, vias 2 -> 6
- net Net-(C55-Pad2): track 61.5 -> 0.00 mm, vias 4 -> 0
- net Net-(C1-Pad2): track 63.5 -> 19.0 mm, vias 3 -> 1
- net Net-(C55-Pad1): track 11.9 -> 0.00 mm
- net Net-(R66-Pad2): track 8.13 -> 0.00 mm
- net Net-(IC13-Pad2): track 7.40 -> 0.00 mm
- net GND: track 977.1 -> 969.8 mm, vias 29 -> 28
- net Net-(R76-Pad2): track 84.9 -> 81.7 mm
- net laag_11: track 449.8 -> 446.8 mm
- net laag_12: track 472.2 -> 469.3 mm
- net laag_10: track 426.6 -> 423.8 mm
- net laag_4: track 360.1 -> 357.4 mm
- net laag_9: track 403.7 -> 400.9 mm
- net laag_8: track 388.8 -> 386.1 mm
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Other:
- board outline added: 380.2 x 220.2 mm
- board text added: "JLCJLCJLCJLC"
